File: Eagle files/EEZ CF-DIC r3B7.sch (EAGLE design)
At the start: 247 parts, among them IC1 MC79L05, IC10 LM211PWR, IC2 LP2951, IC3 VIPer35L, IC4 SI8233BB-D-IS1, IC5 LM5041B, IC6 IR11688STRPBF, IC7 TL072, IC8 TL103W, IC9 TL431, P1 T910W-50K, Q1 BCP56-16.115, Q2 C3M0280090D, Q3 C3M0280090D, Q4 C3M0280090D, Q5 C3M0280090D, Q6 MMBT5401, Q7 IRFS4321PBF, Q8 IRFS4321PBF, X1 B2B-ZR, X2 39-30-1039, X3 90136-1208, X4 39-28-1023

Commit message: r3B7 files without updated BOM
Parts:
- added C76: N.C., rcl:C-EUC0805
- added D24, D25: 1N5819HW-7-F, diode:DIODE-SOD323-W
- added LED2: LTST-C170KRKT, EEZ_Lib1:LED0805
- added OK3: TLP291-GB.SE-T, EEZ_Lib1:TLP291
- added Q9: IRFS4321PBF, EEZ_Lib1:N-MOSFETTO263
- added R85, R86: N.C., rcl:R-EU_R0805
- added X5: 39-28-1023, EEZ_Lib1:MINIFIT_5566-02A
- C4: value N.C. -> CY1Y-470P; device rcl:C-EUC0603 -> EEZ_Lib1:C-EUCY
- C52: value UPW1J152MHD -> 100n; device EEZ_Lib1:ECAP7.5G_18MM -> rcl:C-EUC0603
- C53: value UPW1J152MHD -> N.C.; device EEZ_Lib1:ECAP7.5G_18MM -> rcl:C-EUC0603
- C55: value 1u/100V -> UPW1J152MHD; device rcl:C-EUC1206 -> EEZ_Lib1:ECAP7.5G_18MM
- C56: value HHXC630ARA330MHA0G -> UPW1J152MHD; device Panasonic-EEEFK_EEEFP:EEE-FK1J470P-CASE-F -> EEZ_Lib1:ECAP7.5G_18MM; MPN EEE-FK1J470P -> (none); OC_FARNELL 9696032 -> (none); OC_NEWARK 96K9403 -> (none); PACKAGE CASE-F -> (none); SUPPLIER PANASONIC -> (none); TOLERANCE ±20 % -> (none); VALUE 47UF -> (none); VOLTAGERATING 63 V -> (none)
- C57: value HHXC630ARA330MHA0G -> 1u/100V; device Panasonic-EEEFK_EEEFP:EEE-FK1J470P-CASE-F -> rcl:C-EUC1206
- C58: value 1u/100V -> HHXC630ARA330MHA0G; device rcl:C-EUC1206 -> Panasonic-EEEFK_EEEFP:EEE-FK1J470P-CASE-F; MPN (none) -> EEE-FK1J470P; OC_FARNELL (none) -> 9696032; OC_NEWARK (none) -> 96K9403; PACKAGE (none) -> CASE-F; SUPPLIER (none) -> PANASONIC; TOLERANCE (none) -> ±20 %; VALUE (none) -> 47UF; VOLTAGERATING (none) -> 63 V
- C59: value 100n/100V -> HHXC630ARA330MHA0G; device rcl:C-EUC0805 -> Panasonic-EEEFK_EEEFP:EEE-FK1J470P-CASE-F
- C6: value CY1Y-470P -> N.C.; device EEZ_Lib1:C-EUCY -> rcl:C-EUC0603
- C60: value N.C. -> 1u/100V
- C61: value 4n7/200V -> 100n/100V; device rcl:C-EUC1206 -> rcl:C-EUC0805
- C62: value 100n -> N.C.; device rcl:C-EUC0603 -> rcl:C-EUC1206
- C63: value 10u -> 4n7/200V; device rcl:C-EUC1210 -> rcl:C-EUC1206
- C65: value 4n7/200V -> 10u; device rcl:C-EUC1206 -> rcl:C-EUC1210
- C67: value 100n -> 4n7/200V; device rcl:C-EUC0603 -> rcl:C-EUC1206
- C68, C69: value 100p -> 100n; device rcl:C-EUC0805 -> rcl:C-EUC0603
- C70: value 33n -> 100p
- C71: value 4u7 -> 100p; device EEZ_Lib1:ECAP1206 -> rcl:C-EUC0805
- C72: value 1u -> 33n
- C73: value N.C. -> 4u7; device rcl:C-EUC0805 -> EEZ_Lib1:ECAP1206
- C74: value N.C. -> 1u
- C75: value 100n -> N.C.; device rcl:C-EUC0603 -> rcl:C-EUC0805
- D13, D18, D19: device EEZ_Lib1:SCHOTTKY-2 -> EEZ_Lib1:SCHOTTKY-SIC
- D20, D21: value 1N5819HW-7-F -> BAS316; device diode:DIODE-SOD323-W -> EEZ_Lib1:DIODESOD323R
- IC10: value LM211PWR -> TL431; device EEZ_Lib1:LM211 -> EEZ_Lib1:TL431
- IC6: value IR11688STRPBF -> LM258D; device EEZ_Lib1:IR11688 -> EEZ_Lib1:TL072SOIC8
- IC7: value TL072 -> IR11688STRPBF; device EEZ_Lib1:TL072SOIC8 -> EEZ_Lib1:IR11688
- IC8: value TL103W -> TL072; device EEZ_Lib1:TL103W -> EEZ_Lib1:TL072SOIC8
- IC9: value TL431 -> TL103W; device EEZ_Lib1:TL431 -> EEZ_Lib1:TL103W
- P1: device pot:TRIM_EU-S64W -> EEZ_Lib1:TPOT-S64W
- Q5: value C3M0280090D -> NYC0102BLT1G; device EEZ_Lib1:IRFP240 -> EEZ_Lib1:NYC0102BLT1G
- Q6: value MMBT5401 -> C3M0280090D; device transistor:BC857B-PNP-SOT23-BEC -> EEZ_Lib1:IRFP240
- Q7: value IRFS4321PBF -> MMBT5401; device EEZ_Lib1:N-MOSFETTO263 -> transistor:BC857B-PNP-SOT23-BEC
- R13: value 5K1 -> 470R
- R14: value 470R -> 5K1
- R2: value 120R -> 220K; device rcl:R-EU_R0805 -> rcl:R-EU_R1206
- R3: value 220K -> 120R; device rcl:R-EU_R1206 -> rcl:R-EU_R0805
- R35: value 10R -> 220K; device rcl:R-EU_R0805 -> rcl:R-EU_R1206
- R37: value 47K -> 10R
- R38: value 220K -> 47K; device rcl:R-EU_R1206 -> rcl:R-EU_R0805
- R39: value 1R -> 1K
- R40: value 22R/2W -> 1R; device rcl:R-EU_R2512 -> rcl:R-EU_R0805
- R42: value 100K -> 22R/2W; device rcl:R-EU_R0805 -> rcl:R-EU_R2512
- R43: value 10R -> 100K
- R44: value 1K -> 10R
- R45: value 6K8 -> 1K
- R46: value 22R -> 6K8
- R48: value 30K -> 22R
- R49: value 82K -> 1K
- R50: value 6K8 -> 30K
- R51: value 1K -> 82K
- R53: value N.C. -> 1K
- R54: value 100R -> 6K8
- R55: device rcl:R-EU_R1210 -> rcl:R-EU_R0805
- R56: value 22R/3W -> 3K9; device rcl:R-EU_R2512 -> rcl:R-EU_R0805
- R57: value 22R/3W -> 1K; device rcl:R-EU_R2512 -> rcl:R-EU_R0805
- R58: value 3R3 -> 27K
- R59: value 10R -> 10K
- R60: value 47K -> 100R
- R61: value 3R3 -> N.C.; device rcl:R-EU_R0805 -> rcl:R-EU_R1210
- R64: value 10K -> 3R3
- R65: value 316K -> 10R
- R66: value 10K -> 47K
- R67: value 750R -> 3R3
- R68: value 0R -> 22R/3W; device rcl:R-EU_R0805 -> rcl:R-EU_R2512
- R69: value 750R -> 22R/3W; device rcl:R-EU_R0805 -> rcl:R-EU_R2512
- R70: value 470R -> 10K
- R71: value 12K -> 316K
- R72: value 3K3 -> 10K
- R74: value 30K -> 0R
- R75: value 10K -> 750R
- R76: value 16K -> 470R
- R77: value 220R -> 12K
- R78: value N.C. -> 3K3
- R79: value N.C. -> 750R
- R80: value 3K9 -> 30K
- R81: value 82K -> 10K
- R82: value 27K -> 16K
- R83: value N.C. -> 220R
- R84: value 10K -> N.C.
- X4: value 39-28-1023 -> B2B-ZR; device EEZ_Lib1:MINIFIT_5566-02A -> EEZ_Lib1:B2B-ZR
- renumbered C5A to C4A, C6A to C2A
Connections:
- removed net N$136: LED1.C, R14.1
- removed net N$34: IC10A.-IN, NTC1.P$2, R84.2
- removed net N$65: C48.2, IC5.REF, R35.1, R50.1
- new net +5VREF: C48.2, C53.1, IC5.REF, NTC1.P$1, R36.1, R52.1, R56.2, X4-1.1
- new net N$100: Q5.G, R49.1
- new net N$11: LED1.A, R13.2
- new net N$126: D20.C, D21.C, Q5.A
- new net N$130: D20.A, LED2.C
- new net N$16: LED2.A, R39.2
- new net N$26: IC6B.-IN, R56.1, R58.1
- new net N$32: OK2.C, R39.1
- new net N$38: IC6B.OUT, R49.2, R57.1
- new net N$42: IC6A.-IN, IC6A.OUT, IC6B.+IN
- net +12V: now also C52.1, C6.1, IC6P.V+, OK2.A, R37.2, R44.2; no longer C4.1, R36.2, R43.2
- net +2.5VREF: now also C74.1, IC9-1.+IN1, R72.2, R78.1; no longer C72.1, IC8-1.+IN1, NTC1.P$1, R66.2, R72.1, R80.2
- net +6V: now also R13.1, R65.1; no longer LED1.A, R59.1
- net 0V: now also C6.2, Q6.S, R38.2, R40.1, R40.2; no longer C4.2, Q5.S, R37.2, R39.1, R39.2
- net AGND: now also C52.2, C53.2, IC6P.V-, OK3.EMIT, Q5.C, Q7.C, R46.2, R50.2, R51.2, R54.2, R57.2, R58.2, R59.2; no longer OK2.EMIT, Q6.C, R45.2, R48.2, R49.2, R52.2
- net CLAMP_C: now also R42.1; no longer R40.1
- net CT_OUT: now also R53.1; no longer R51.1
- net DC_BUS: now also R35.1, R42.2; no longer R38.1, R40.2
- net FB: now also C75.2, IC10.REF, R77.1, R81.2, R82.2, R85.2, R86.2; no longer C73.2, IC9.REF, R71.1, R75.2, R76.2, R79.2, R83.2
- net GND: now also C55.-, C56.-, C60.2, C62.1, C68.2, C69.2, C73.-, C74.2, IC10.A, IC7.GND, IC7.VS, IC8A.+IN, IC8B.+IN, IC9-1.VCC-, LED1.C, OK2.EMIT, Q9.S, R66.2, R86.1, X5-2.1; no longer C52.-, C53.-, C55.2, C56.2, C60.1, C62.2, C71.-, C72.2, C75.2, IC10A.E, IC10P.V-, IC6.GND, IC6.VS, IC7A.+IN, IC7B.+IN, IC8-1.VCC-, IC9.A, Q7.S, R13.2, R60.2, R82.2, R83.1, R84.1, X4-2.1
- net ISO_FB: now also OK3.COL, Q7.E, R55.1; no longer OK2.COL, Q6.E, R53.1
- net L_PULL: now also Q6.D; no longer Q5.D
- net N$1: now also C70.2, IC8A.-IN, R74.2, R75.1, R79.1; no longer C68.2, IC7A.-IN, R68.2, R69.1, R73.1
- net N$10: now also C71.2, IC9-1.-IN1, R80.1, R81.1; no longer C69.2, IC8-1.-IN1, R74.1, R75.1
- net N$101: now also R14.1; no longer R13.1
- net N$12: now also R71.1, R77.2; no longer R65.1, R71.2
- net N$13: now also D22.C, R47.1; no longer D20.C, R46.1
- net N$132: now also IC8B.-IN, R70.2, R72.1; no longer IC7B.-IN, R64.2, R66.1
- net N$134: now also C70.1, IC8A.OUT, R83.2; no longer C68.1, IC7A.OUT, R77.2
- net N$14: now also D23.C, Q6.G, R48.1; no longer D21.C, Q5.G, R47.1
- net N$140: now also R3.2; no longer R2.2
- net N$15: now also C5.2; no longer C6.2
- net N$17: now also C76.2, R85.1; no longer C74.2, R79.1
- net N$18: now also IC7.MOT, R66.1; no longer IC6.MOT, R60.1
- net N$19: now also R51.1; no longer R49.1
- net N$2: now also R35.2, R43.1; no longer R38.2, R42.1
- net N$22: now also R50.1; no longer R48.1
- net N$24: now also C4.2; no longer C5.2
- net N$25: now also R45.1; no longer R44.1
- net N$27: now also R3.1; no longer R2.1
- net N$29: now also R38.1; no longer R37.1
- net N$30: now also R2.2; no longer R3.2
- net N$33: now also R2.1; no longer R3.1
- net N$35: now also R55.2; no longer R53.2
- net N$37: now also R53.2; no longer R51.2
- net N$47: now also Q7.B, R52.2, R54.1; no longer Q6.B, R50.2, R52.1
- net N$53: now also IC8B.OUT, R70.1, R75.2; no longer IC7B.OUT, R64.1, R69.2
- net N$54: now also R44.1; no longer R43.1
- net N$57: now also IC9-2.+IN; no longer IC8-2.+IN
- net N$6: now also C64.1, C65.1, IC7.VCC, R65.2; no longer C62.1, C63.1, IC6.VCC, R59.2
- net N$63: now also R37.1; no longer R36.1
- net N$64: now also R73.2, R74.1; no longer R67.2, R68.1
- net N$66: now also C63.1, R62.2, R63.2; no longer C61.1, R56.2, R57.2
- net N$67: now also C67.1, R68.2, R69.2; no longer C65.1, R62.2, R63.2
- net N$7: now also IC6A.+IN, NTC1.P$2, R59.1, X4-2.1; no longer IC10A.+IN, R80.1, R81.2, R82.1
- net N$74: now also D24.C, IC7.GATE1, R64.2; no longer D22.C, IC6.GATE1, R58.2
- net N$75: now also D25.C, IC7.GATE2, R67.2; no longer D23.C, IC6.GATE2, R61.2
- net N$76: now also C71.1, C72.1, C75.1, C76.1, IC10.C, IC9-1.OUT1, OK3.C, R84.2; no longer C69.1, C70.1, C73.1, C74.1, IC8-1.OUT1, IC9.C, OK2.C, R78.2
- net N$8: now also C62.2, R61.1; no longer C60.2, R55.1
- net N$9: now also C72.2, R80.2; no longer C70.2, R74.2
- net NFB_OFFSET: now also C73.+, R73.1, R82.1, R83.1; no longer C71.+, R67.1, R76.1, R77.1
- net OK_A: now also OK3.A, R76.1, R84.1; no longer OK2.A, R70.1, R78.1
- net PE: now also C4.1; no longer C6.1
- net POUT+: now also C55.+, C56.+, C57.1, R60.1, R71.2; no longer C52.+, C53.+, C55.1, R54.1, R65.2
- net PREG_OUT+: now also C60.1, C61.1, R60.2, R61.2, X5-1.1; no longer C56.1, C57.1, R54.2, R55.2, X4-1.1
- net PULL: now also D23.A, R48.2; no longer D21.A, R47.2
- net PUSH: now also D22.A, R47.2; no longer D20.A, R46.2
- net PWRGOOD: now also OK2.COL; no longer IC10A.C, R81.1
- net REF: now also R36.2; no longer R35.2
- net S1_DOT_OUT: now also IC7.VD1, Q8.D, R62.1, R63.1; no longer IC6.VD1, Q7.D, R56.1, R57.1
- net S2_OUT: now also IC7.VD2, Q9.D, R68.1, R69.1; no longer IC6.VD2, Q8.D, R62.1, R63.1
- net SR_OUT1: now also D24.A, Q8.G, R64.1; no longer D22.A, Q7.G, R58.1
- net SR_OUT2: now also D25.A, Q9.G, R67.1; no longer D23.A, Q8.G, R61.1
- net ULVO: now also D21.A, R43.2, R45.2, R46.1; no longer R42.2, R44.2, R45.1
- net U_MON1: now also IC9-2.-IN, IC9-2.OUT, R79.2; no longer IC8-2.-IN, IC8-2.OUT, R73.2
- net V+: now also C66.1, C69.1, IC8P.V+, IC9-1.VCC+, R76.2, R78.2; no longer C64.1, C67.1, C75.1, IC10P.V+, IC7P.V+, IC8-1.VCC+, R70.2, R72.2
- net V-: now also C68.1, IC8P.V-; no longer C66.1, IC7P.V-
Other:
- note added: ""Fault" (red)"
- note added: ""Power" (yellow)"
- note added: "(optional)"
- note added: "-5 Vdc 7"
- note added: "More info at https://www.envox.hr/eez"
- note added: "Optional NFB if tracker is not used!"
- note added: "Thermal protection"
- note removed: "+5 Vdc 7"
- note removed: "More info at http://www.envox.hr/eez"
- note removed: "Temperature alarm (optional)"
- moved on the sheet: C10, C11, C12, C13, C14, C15, C16, C17, C18, C19, C20, C21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
