File: Eagle files/EEZ CF-DIC r3B8.sch (EAGLE design)
At the start: 256 parts, among them IC1 MC79L05, IC10 TL431, IC2 LP2951, IC3 VIPer35L, IC4 SI8233BB-D-IS1, IC5 LM5041B, IC6 LM258D, IC7 IR11688STRPBF, IC8 TL072, IC9 TL103W, P1 T910W-50K, Q1 BCP56-16.115, Q2 C3M0280090D, Q3 C3M0280090D, Q4 C3M0280090D, Q5 NYC0102BLT1G, Q6 C3M0280090D, Q7 MMBT5401, Q8 IRFS4321PBF, Q9 IRFS4321PBF, X1 B2B-ZR, X2 39-30-1039, X3 90136-1208, X4 B2B-ZR, X5 39-28-1023

Commit message: first r3B8 version (no BOM)
Parts:
- removed TP8: (no value), EEZ_Lib1:PCB_TEST_TABSHIELD
- added R87: N.C., rcl:R-EU_R0805
- C10: value EEEFK1V470P -> 1n/1kV; device EEZ_Lib1:ECAPPANASONIC_H -> rcl:C-EUC1210
- C11: value 1u -> EEEFK1V470P; device rcl:C-EUC0805 -> EEZ_Lib1:ECAPPANASONIC_H
- C12: value 1n/1kV -> 1u; device rcl:C-EUC1210 -> rcl:C-EUC0805
- C18: value 3n3 -> CY1Y-470P; device rcl:C-EUC0805 -> EEZ_Lib1:C-EUCY
- C19: value CY1Y-470P -> 3n3; device EEZ_Lib1:C-EUCY -> rcl:C-EUC0805
- C24: value 470u -> WL1C158M12020BB
- C27: value 100p -> 2n2
- C28: value 2n2 -> 100p
- C3: value 3n3 -> 1n
- C6: value N.C. -> 100n
- C7: value EEEFK1V470P -> WL1E337M1012MBB
- D3: value 1N5819HW-7-F -> US1M-DIO; device diode:DIODE-SOD323-W -> EEZ_Lib1:DIODEDO214AA
- D4: value US1K-DIO -> SKL16; device EEZ_Lib1:DIODEDO214AA -> EEZ_Lib1:SCHOTTKYSOD123
- D6, D7, D9: value 1N5819HW-7-F -> SKL16; device diode:DIODE-SOD323-W -> EEZ_Lib1:SCHOTTKYSOD123
- IC2: value LP2951 -> LP2951SO8
- IC3: value VIPer35L -> VIPER35
- L2, L3, L4: device EEZ_inductors_and_transformers:DE0403 -> EEZ_Lib1:DE0403
- R11: value 120R -> 33R
- R12: value 16K -> ***
- R13: value 470R -> 120R
- R14: value 5K1 -> 16K
- R15: value 10K -> 47K
- R16: value N.C. -> 750R
- R17: value 47K -> 5K1
- R18: value 750R -> 470R
- R19: value 12K -> 10K
- R21: value 47K -> 12K
- R22, R39: value 1K -> 47K
- R23: value 10K -> 1K
- R24: value 6R2 -> 10K
- R25: value N.C. -> 6R2
- R26: value 10R -> N.C.
- R28: value 100R -> 10R
- R29, R31: value 22R/2W -> 100R; device rcl:R-EU_R2512 -> rcl:R-EU_R0805
- R3: value 120R -> ???
- R30: value 100R -> 22R/2W; device rcl:R-EU_R0805 -> rcl:R-EU_R2512
- R32: value 1R -> 22R/2W; device rcl:R-EU_R0805 -> rcl:R-EU_R2512
- R33: value 30K -> 1R
- R34: value 10R -> 30K
- R35: value 220K -> 10R; device rcl:R-EU_R1206 -> rcl:R-EU_R0805
- R36: value 10R -> 220K; device rcl:R-EU_R0805 -> rcl:R-EU_R1206
- R38, R66: value 47K -> 10R
- R4: value 22R -> 1K8
- R40: value 1R -> 1K
- R41: value 22R/2W -> 1R; device rcl:R-EU_R2512 -> rcl:R-EU_R0805
- R43: value 100K -> 22R/2W; device rcl:R-EU_R0805 -> rcl:R-EU_R2512
- R44: value 10R -> 100K
- R45: value 1K -> 10R
- R46, R54: value 6K8 -> 1K
- R47: value 22R -> 6K8
- R49: value 1K -> 22R
- R5: value 1K8 -> 120R
- R50: value 30K -> 1K
- R51: value 82K -> 30K
- R52: value 6K8 -> 82K
- R53: value 1K -> 6K8
- R55: value N.C. -> 6K8
- R56: value 3K9 -> N.C.
- R57: value 1K -> 3K9
- R58: value 27K -> 1K
- R59: value 10K -> 27K
- R6: value 120R -> 220K; device rcl:R-EU_R0805 -> rcl:R-EU_R1206
- R60: value 100R -> 10K
- R61: value N.C. -> 100R; device rcl:R-EU_R1210 -> rcl:R-EU_R0805
- R62: value 22R/3W -> N.C.; device rcl:R-EU_R2512 -> rcl:R-EU_R1210
- R64: value 3R3 -> 22R/3W; device rcl:R-EU_R0805 -> rcl:R-EU_R2512
- R65: value 10R -> 3R3
- R67: value 3R3 -> 47K
- R68: value 22R/3W -> 3R3; device rcl:R-EU_R2512 -> rcl:R-EU_R0805
- R7, R8: value 220K -> 33K; device rcl:R-EU_R1206 -> rcl:R-EU_R1210
- R70: value 10K -> 22R/3W; device rcl:R-EU_R0805 -> rcl:R-EU_R2512
- R71: value 316K -> 10K
- R72: value 10K -> 316K
- R73: value 750R -> 10K
- R74: value 0R -> 750R
- R75: value 750R -> 0R
- R76: value 470R -> 750R
- R77: value 12K -> 470R
- R78: value 3K3 -> 12K
- R79: value 750R -> 3K3
- R80: value 30K -> 750R
- R81: value 10K -> 30K
- R82: value 16K -> 10K
- R83: value 220R -> 16K
- R84: value N.C. -> 220R
- TP6: device EEZ_Lib1:PCB_TEST_TABSHIELD -> EEZ_Lib1:TEST_POINT-2
- TP7: device EEZ_Lib1:TEST_POINT-2 -> EEZ_Lib1:PCB_TEST_TABSHIELD
- TR1: device EEZ_inductors_and_transformers:FERYSTER_5572 -> EEZ_Lib1:FERYSTER_5572
- ZD1: value BZT52C20-DC -> BZX384-C13; device EEZ_Lib1:ZENER-DIODESOD123FL -> EEZ_Lib1:ZENER-DIODESOD323
- ZD2: value BZX384-C13 -> BZT52C20-DC; device EEZ_Lib1:ZENER-DIODESOD323 -> EEZ_Lib1:ZENER-DIODESOD123
- ZD3: value MMSZ5V1T1G -> MMSZ5230BT1G
Connections:
- removed net +15V_REC: C10.+, D2.C, L2.1, R6.1
- removed net -7V_REC: C14.-, D5.A, L3.1, R10.1
- removed net 15VAC: C9.2, D2.A, TR1.S3_DOT
- removed net AUX: C3.2, D1.A, D10.A, R16.2, TR1.S_BIAS_DOT
- removed net AUX_OUT: C20.2, C7.+, IC3.VDD, Q1.C, R4.2, R5.1, ZD1.C
- removed net FB2: OK1.C, R22.1, ZD3.C
- removed net N$101: IC2.FB, R12.2, R14.1
- removed net N$11: LED1.A, R13.2
- removed net N$133: C8.1, Q1.B, R5.2, ZD2.C
- removed net N$135: OK1.A, R18.2
- removed net N$137: C12.2, D4.C, R7.2
- removed net N$138: C26.2, C28.1, IC3.FB, OK1.COL
- removed net N$139: C9.1, R6.2
- removed net N$141: C27.1, IC3.ZCD, R16.1, R17.1, R19.2
- removed net N$144: C18.1, R10.2
- removed net N$146: C21.1, R11.2
- removed net N$152: C26.1, R21.1
- removed net N$155: D10.C, D11.C, R17.2
- removed net N$27: D1.C, R3.1, R4.1
- removed net N$4: C19.1, JP2.COM
- removed net N$49: R8.2, R9.1
- new net +15V: D2.A, R5.1, TR1.S3_DOT
- new net +15V_REC2: C11.+, C9.2, D2.C, L2.1
- new net -7V_REC2: C14.-, C19.2, D5.A, L3.1
- new net AUX_AC: D1.A, D10.A, R12.2, R3.1, TR1.S_BIAS_DOT
- new net AUX_DC: C3.2, C7.+, D1.C, Q1.C, R11.1, R4.1
- new net FB3: OK1.C, R23.1, ZD3.C
- new net N$103: C18.1, JP2.COM
- new net N$104: C26.1, R22.1
- new net N$106: D10.C, D11.C, R15.2
- new net N$108: R6.2, R9.1
- new net N$87: IC2.FB, R14.2, R17.1
- new net N$88: C8.1, Q1.B, R4.2, ZD1.C
- new net N$89: OK1.A, R16.2
- new net N$90: LED1.C, R18.1
- new net N$91: C10.2, D3.C, R8.2
- new net N$92: C26.2, C27.1, IC3.FB, OK1.COL
- new net N$93: C9.1, R5.2
- new net N$95: C28.1, IC3.ZCD, R12.1, R15.1, R21.2
- new net N$96: R7.2, R8.1
- new net N$97: C19.1, R10.2
- new net N$98: C21.1, R13.2
- new net VIPER_VDD: C20.1, IC3.VDD, R11.2, ZD2.C
- net +12V: now also R27.2, R38.2, R45.2; no longer R26.2, R37.2, R44.2
- net +2.5VREF: now also R73.2, R79.1; no longer R72.2, R78.1
- net +5VREF: now also R37.1, R53.1, R57.2; no longer R36.1, R52.1, R56.2
- net +6V: now also LED1.A, R23.2, R66.1; no longer R13.1, R22.2, R65.1
- net +6V_REC: now also C21.2, R16.1; no longer R11.1, R18.1
- net -15V: now also C11.-, C12.2, X3-2.S; no longer C10.-, C11.2
- net 0V: now also C20.2, JP2.NO, R21.1, R22.2, R39.2, R41.1, R41.2, TP3.P$1; no longer C20.1, JP2.NC, R19.1, R21.2, R38.2, R40.1, R40.2, TP1.P$1, TP4.P$1
- net 6VAC: now also R13.1; no longer C21.2
- net 7VAC: now also R10.1; no longer C18.2
- net AGND: now also R26.2, R33.2, R34.1, R47.2, R52.2, R55.2, R60.2; no longer R23.2, R32.1, R32.2, R46.2, R50.2, R54.2, R57.2
- net BUCK_OUT: now also TP2.P$1; no longer TP3.P$1
- net CLAMP_C: now also R43.1; no longer R41.1
- net CT_OUT: now also R26.1, R54.1; no longer R24.1, R53.1
- net DC_BUS: now also C10.1, R36.1, R43.2, R6.1; no longer C12.1, R35.1, R41.2, R8.1
- net DC_OUT: now also C12.1; no longer C11.1
- net FB: now also R78.1, R83.2, R87.2, TP7.P$1; no longer R77.1, R81.2, R85.2, TP8.P$1
- net GND: now also C18.2, D4.C, R17.2, R18.2, R67.2, R87.1, TP1.P$1, TP6.GND; no longer C19.2, D3.C, LED1.C, R14.2, R66.2, R86.1, TP2.P$1, TP7.GND
- net HD: now also R29.2; no longer R28.2
- net HI_OUT: now also R28.2; no longer R27.2
- net ISO_FB: now also R56.1, TP5.P$1; no longer R55.1, TP6.P$1
- net LD: now also R31.2; no longer R30.2
- net LO_OUT: now also R35.1; no longer R34.1
- net L_PUSH: now also R30.2; no longer R29.2
- net N$1: now also R75.2, R76.1, R80.1; no longer R74.2, R75.1, R79.1
- net N$10: now also R82.1; no longer R80.1
- net N$100: now also R50.1; no longer R49.1
- net N$12: now also R72.1, R78.2; no longer R71.1, R77.2
- net N$13: now also R48.1; no longer R47.1
- net N$132: now also R71.2, R73.1; no longer R70.2, R72.1
- net N$134: now also R84.2; no longer R83.2
- net N$14: now also R49.1; no longer R48.1
- net N$16: now also R40.2; no longer R39.2
- net N$17: now also R86.1; no longer R85.1
- net N$18: now also R67.1; no longer R66.1
- net N$19: now also R52.1; no longer R51.1
- net N$2: now also R36.2, R44.1; no longer R35.2, R43.1
- net N$21: now also R28.1; no longer R27.1
- net N$22: now also R51.1; no longer R50.1
- net N$25: now also R46.1; no longer R45.1
- net N$26: now also R57.1, R59.1; no longer R56.1, R58.1
- net N$29: now also R35.2, R39.1; no longer R34.2, R38.1
- net N$31: now also R27.1; no longer R26.1
- net N$32: now also R40.1; no longer R39.1
- net N$35: now also R56.2; no longer R55.2
- net N$36: now also R29.1; no longer R28.1
- net N$37: now also R54.2; no longer R53.2
- net N$38: now also R50.2, R58.1; no longer R49.2, R57.1
- net N$40: now also R31.1; no longer R30.1
- net N$41: now also R30.1, R32.2; no longer R29.1, R31.2
- net N$47: now also R53.2, R55.1; no longer R52.2, R54.1
- net N$48: now also R34.2; no longer R33.2
- net N$5: now also R32.1; no longer R31.1
- net N$50: now also R24.1; no longer R23.1
- net N$53: now also R71.1, R76.2; no longer R70.1, R75.2
- net N$54: now also R45.1; no longer R44.1
- net N$6: now also R66.2; no longer R65.2
- net N$63: now also R38.1; no longer R37.1
- net N$64: now also R74.2, R75.1; no longer R73.2, R74.1
- net N$66: now also R64.2; no longer R62.2
- net N$67: now also R70.2; no longer R68.2
- net N$7: now also R60.1; no longer R59.1
- net N$74: now also R65.2; no longer R64.2
- net N$75: now also R68.2; no longer R67.2
- net N$76: now also R85.2; no longer R84.2
- net N$8: now also R62.1; no longer R61.1
- net N$9: now also R81.2; no longer R80.2
- net NFB_OFFSET: now also R74.1, R84.1; no longer R73.1, R82.1
- net OK_A: now also R77.1, R85.1; no longer R76.1, R84.1
- net PE: now also JP2.NC; no longer JP2.NO
- net POUT+: now also R61.1, R72.2; no longer R60.1, R71.2
- net PREG_OUT+: now also R62.2, TP6.TIP; no longer R60.2, TP7.TIP, X3-2.S
- net PULL: now also R49.2; no longer R48.2
- net PUSH: now also R48.2; no longer R47.2
- net PWRGOOD: now also R19.2; no longer R15.2
- net REF: now also R37.2; no longer R36.2
- net S1_DOT_OUT: now also R64.1; no longer R62.1
- net S2_OUT: now also R70.1; no longer R68.1
- net SR_OUT1: now also R65.1; no longer R64.1
- net SR_OUT2: now also R68.1; no longer R67.1
- net ULVO: now also R44.2, R46.2, R47.1, TP4.P$1; no longer R43.2, R45.2, R46.1, TP5.P$1
- net U_MON1: now also R80.2; no longer R79.2
- net V+: now also R14.1, R19.1, R77.2, R79.2; no longer R12.1, R15.1, R76.2, R78.2
- net V-: now also D4.A; no longer D3.A
- net VIPER_D: now also D3.A; no longer D4.A
Other:
- note added: "18p"
- note added: "5R1 (4R7)"
- note added: "LM5041B Vcc"
- note added: "N.C."
- note added: "Post-regulator pass mosfet Drain"
- note added: "Post-regulator pass mosfet Vbias"
- note added: "US1K-DIO"
- note added: "V+ for sync rectifier gate driver"
- note added: "V- for downprogrammer"
- note removed: ""Power" (yellow)"
- note removed: "Cfb"
- note removed: "Cfb1"
- note removed: "Rfb1"
- moved on the sheet: C12, C13, C14, C15, C16, C17, C18, C19, C20, C21, C22, C23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
