File: Eagle files/EEZ CF-DIC r4B4.sch (EAGLE design)
At the start: 256 parts, among them IC1 MC79L05, IC10 TL431, IC2 LP2951SO8, IC3 VIPER35, IC4 SI8233BB-D-IS1, IC5 LM5041B, IC6 LM258D, IC7 IR11688STRPBF, IC8 TL072, IC9 TL103W, P1 T910W-50K, Q1 BCP56-16.115, Q2 C3M0280090D, Q3 C3M0280090D, Q4 C3M0280090D, Q5 NYC0102BLT1G, Q6 C3M0280090D, Q7 MMBT5401, Q8 IRFS4321PBF, Q9 IRFS4321PBF, X1 B2B-ZR, X2 39-30-1039, X3 90136-1208, X4 B2B-ZR, X5 39-28-1023

Commit message: r4B4 with updated BOM
Parts:
- removed C2A: N.C., EEZ_Lib1:C-EUCY
- removed C72: 33n, rcl:C-EUC0805
- removed C73: 4u7, EEZ_Lib1:ECAP1206
- removed C74: 1u, rcl:C-EUC0805
- removed C75, C76: N.C., rcl:C-EUC0805
- removed D23, D24, D25: 1N5819HW-7-F, diode:DIODE-SOD323-W
- removed IC10: TL431, EEZ_Lib1:TL431
- removed IC8: TL072, EEZ_Lib1:TL072SOIC8
- removed IC9: TL103W, EEZ_Lib1:TL103W
- removed JP4: JP3-CUT, EEZ_Lib1:JP3-CUT
- removed NTC1: 10K/3570K, EEZ_Lib1:NTCR_0805
- removed Q9: IRFS4321PBF, EEZ_Lib1:N-MOSFETTO263
- removed R78: 12K, rcl:R-EU_R0805
- removed R79: 3K3, rcl:R-EU_R0805
- removed R80: 750R, rcl:R-EU_R0805
- removed R81: 30K, rcl:R-EU_R0805
- removed R82: 10K, rcl:R-EU_R0805
- removed R83: 16K, rcl:R-EU_R0805
- removed R84: 220R, rcl:R-EU_R0805
- removed R85, R86, R87: N.C., rcl:R-EU_R0805
- added C5A: N.C., EEZ_Lib1:C-EUCY
- C10: value 1n/1kV -> EEEFK1V470P; device rcl:C-EUC1210 -> EEZ_Lib1:ECAPPANASONIC_H
- C11: value EEEFK1V470P -> 1u; device EEZ_Lib1:ECAPPANASONIC_H -> rcl:C-EUC0805
- C12: value 1u -> 1n/1kV; device rcl:C-EUC0805 -> rcl:C-EUC1210
- C16: value 470n -> 3n3
- C17: value 100n -> CY1Y-470P; device rcl:C-EUC0603 -> EEZ_Lib1:C-EUCY
- C18: value CY1Y-470P -> 100n; device EEZ_Lib1:C-EUCY -> rcl:C-EUC0603
- C20: value 100n -> 470u; device rcl:C-EUC0603 -> EEZ_Lib1:ECAP5G_10.5MM
- C21: value 3n3 -> EEEFK1V470P; device rcl:C-EUC0805 -> EEZ_Lib1:ECAPPANASONIC_H
- C22: value 100n -> 4u7; device rcl:C-EUC0603 -> rcl:C-EUC1206
- C23: value 4u7 -> 33n; device EEZ_Lib1:ECAP1206 -> rcl:C-EUC0805
- C24: value WL1C158M12020BB -> 100p; device EEZ_Lib1:ECAP5G_10.5MM -> rcl:C-EUC0805
- C25: value 4u7 -> 2n2; device rcl:C-EUC1206 -> rcl:C-EUC0805
- C26: value 33n -> 1u
- C27: value 2n2 -> 100n; device rcl:C-EUC0805 -> rcl:C-EUC0603
- C28: value 100p -> UCY2G121MHD; device rcl:C-EUC0805 -> EEZ_Lib1:ECAP7.5G_18MM
- C29: value 1u -> UCY2G121MHD; device rcl:C-EUC0805 -> EEZ_Lib1:ECAP7.5G_18MM
- C3: value 1n -> 3n3
- C30, C35, C39: value 100n -> 10n
- C31, C32: value UCY2G121MHD -> 100n; device EEZ_Lib1:ECAP7.5G_18MM -> rcl:C-EUC0603
- C33: value 10n -> 100n/500V; device rcl:C-EUC0603 -> rcl:C-EUC1812
- C36: value 100n/500V -> 100n; device rcl:C-EUC1812 -> rcl:C-EUC0603
- C38: value 10n -> 2n2/1kV; device rcl:C-EUC0603 -> rcl:C-EUC1210
- C40: value 100n -> 1u; device rcl:C-EUC0603 -> rcl:C-EUC0805
- C41: value 2n2/1kV -> 100n; device rcl:C-EUC1210 -> rcl:C-EUC0603
- C42: value 10n -> 1u; device rcl:C-EUC0603 -> rcl:C-EUC0805
- C43: value 1u -> 100n/500V; device rcl:C-EUC0805 -> rcl:C-EUC1812
- C44: value 100n -> 100n/500V; device rcl:C-EUC0603 -> rcl:C-EUC1812
- C45: value 1u -> 100n; device rcl:C-EUC0805 -> rcl:C-EUC0603
- C46: value 100n/500V -> 470p; device rcl:C-EUC1812 -> rcl:C-EUC0805
- C47: value 100n/500V -> 220p; device rcl:C-EUC1812 -> rcl:C-EUC0805
- C48: value 100n -> N.C.; device rcl:C-EUC0603 -> rcl:C-EUC0805
- C49: value 220p -> 100n; device rcl:C-EUC0805 -> rcl:C-EUC0603
- C50: value 470p -> N.C.; device rcl:C-EUC0805 -> rcl:C-EUC0603
- C51: value N.C. -> UPW1J152MHD; device rcl:C-EUC0805 -> EEZ_Lib1:ECAP7.5G_18MM
- C52: value 100n -> UPW1J152MHD; device rcl:C-EUC0603 -> EEZ_Lib1:ECAP7.5G_18MM
- C53: value N.C. -> UPW1J152MHD; device rcl:C-EUC0603 -> EEZ_Lib1:ECAP7.5G_18MM
- C54: value UPW1J152MHD -> 1u/100V; device EEZ_Lib1:ECAP7.5G_18MM -> rcl:C-EUC1206
- C55: value UPW1J152MHD -> HHXC630ARA330MHA0G; device EEZ_Lib1:ECAP7.5G_18MM -> Panasonic-EEEFK_EEEFP:EEE-FK1J470P-CASE-F; MPN (none) -> EEE-FK1J470P; OC_FARNELL (none) -> 9696032; OC_NEWARK (none) -> 96K9403; PACKAGE (none) -> CASE-F; SUPPLIER (none) -> PANASONIC; TOLERANCE (none) -> ±20 %; VALUE (none) -> 47UF; VOLTAGERATING (none) -> 63 V
- C56: value UPW1J152MHD -> HHXC630ARA330MHA0G; device EEZ_Lib1:ECAP7.5G_18MM -> Panasonic-EEEFK_EEEFP:EEE-FK1J470P-CASE-F
- C58: value HHXC630ARA330MHA0G -> 100n/100V; device Panasonic-EEEFK_EEEFP:EEE-FK1J470P-CASE-F -> rcl:C-EUC0805; MPN EEE-FK1J470P -> (none); OC_FARNELL 9696032 -> (none); OC_NEWARK 96K9403 -> (none); PACKAGE CASE-F -> (none); SUPPLIER PANASONIC -> (none); TOLERANCE ±20 % -> (none); VALUE 47UF -> (none); VOLTAGERATING 63 V -> (none)
- C59: value HHXC630ARA330MHA0G -> N.C.; device Panasonic-EEEFK_EEEFP:EEE-FK1J470P-CASE-F -> rcl:C-EUC1206
- C6: value 100n -> N.C.
- C60: value 1u/100V -> 4n7/200V
- C61: value 100n/100V -> 100n; device rcl:C-EUC0805 -> rcl:C-EUC0603
- C62: value N.C. -> 4u7
- C63: value 4n7/200V -> 100n; device rcl:C-EUC1206 -> rcl:C-EUC0603
- C64: value 100n -> 4n7/200V; device rcl:C-EUC0603 -> rcl:C-EUC1206
- C65: value 10u -> 100n; device rcl:C-EUC1210 -> rcl:C-EUC0603
- C67: value 4n7/200V -> 100p; device rcl:C-EUC1206 -> rcl:C-EUC0805
- C68: value 100n -> 100p; device rcl:C-EUC0603 -> rcl:C-EUC0805
- C69: value 100n -> 33n; device rcl:C-EUC0603 -> rcl:C-EUC0805
- C7: value WL1E337M1012MBB -> EEEFK1V470P
- C70: value 100p -> 4u7; device rcl:C-EUC0805 -> EEZ_Lib1:ECAP1206
- C71: value 100p -> 1u
- D10: value BAS316 -> C3D02065E; device EEZ_Lib1:DIODESOD323R -> EEZ_Lib1:SCHOTTKY-SIC
- D11: value BAS316 -> N.C.; device EEZ_Lib1:DIODESOD323R -> diode:DIODE-SOD323-W
- D12: value BAS316 -> C3D03060A; device EEZ_Lib1:DIODESOD323R -> EEZ_Lib1:SCHOTTKY-TO220
- D13, D19: value C3D02065E -> 1N5819HW-7-F; device EEZ_Lib1:SCHOTTKY-SIC -> diode:DIODE-SOD323-W
- D15: value C3D03060A -> C3D02065E; device EEZ_Lib1:SCHOTTKY-TO220 -> EEZ_Lib1:SCHOTTKY-SIC
- D16: value 1N5819HW-7-F -> C3D02065E; device diode:DIODE-SOD323-W -> EEZ_Lib1:SCHOTTKY-SIC
- D17: value N.C. -> BAS316; device diode:DIODE-SOD323-W -> EEZ_Lib1:DIODESOD323R
- D18: value C3D02065E -> BAS316; device EEZ_Lib1:SCHOTTKY-SIC -> EEZ_Lib1:DIODESOD323R
- D20, D21: value BAS316 -> 1N5819HW-7-F; device EEZ_Lib1:DIODESOD323R -> diode:DIODE-SOD323-W
- D3: value US1M-DIO -> US1K-DIO
- D4: value SKL16 -> SS110B; device EEZ_Lib1:SCHOTTKYSOD123 -> EEZ_Lib1:SCHOTTKYSMB
- D6: value SKL16 -> 1N5819HW-7-F; device EEZ_Lib1:SCHOTTKYSOD123 -> diode:DIODE-SOD323-W
- D7, D9: value SKL16 -> BAS316; device EEZ_Lib1:SCHOTTKYSOD123 -> EEZ_Lib1:DIODESOD323R
- D8: value SS110B -> BAS316; device EEZ_Lib1:SCHOTTKYSMB -> EEZ_Lib1:DIODESOD323R
- IC1: value MC79L05 -> VIPer35L; device EEZ_Lib1:MC79LXXSOIC -> EEZ_Lib1:VIPER35
- IC2: value LP2951SO8 -> SI8233BB-D-IS1; device EEZ_Lib1:LP2951SO8 -> EEZ_Lib1:SI8233
- IC3: value VIPER35 -> LM5041B; device EEZ_Lib1:VIPER35 -> EEZ_Lib1:LM5041
- IC4: value SI8233BB-D-IS1 -> LM258D; device EEZ_Lib1:SI8233 -> EEZ_Lib1:TL072SOIC8
- IC5: value LM5041B -> IR11688STRPBF; device EEZ_Lib1:LM5041 -> EEZ_Lib1:IR11688
- IC6: value LM258D -> TL072
- IC7: value IR11688STRPBF -> TL103W; device EEZ_Lib1:IR11688 -> EEZ_Lib1:TL103W
- JP3: value 0R -> JP3-CUT; device rcl:R-EU_R0805 -> EEZ_Lib1:JP3-CUT
- L2, L3, L4: device EEZ_Lib1:DE0403 -> EEZ_inductors_and_transformers:DE0403
- Q1: value BCP56-16.115 -> MMBT5551; device EEZ_Lib1:BCP56 -> transistor:MMBT5551LT1-NPN-SOT23-BEC
- Q2, Q3, Q4, Q6: device EEZ_Lib1:IRFP240 -> EEZ_Lib1:N-MOSFETTO247
- Q7: value MMBT5401 -> IRFS4321PBF; device transistor:BC857B-PNP-SOT23-BEC -> EEZ_Lib1:N-MOSFETTO263
- R11: value 33R -> 470R
- R12: value *** -> 10K
- R13: value 120R -> N.C.
- R14: value 16K -> 47K
- R15: value 47K -> 750R
- R16: value 750R -> 12K
- R17: value 5K1 -> 1K8
- R18: value 470R -> 47K
- R19: value 10K -> 1K
- R20: value 1K8 -> 10K
- R21: value 12K -> 6R2
- R22: value 47K -> N.C.
- R23: value 1K -> 10R
- R24, R60: value 10K -> 10R
- R25: value 6R2 -> 100R
- R26: value N.C. -> 22R/2-3W; device rcl:R-EU_R0805 -> rcl:R-EU_R2512
- R27: value 10R -> 100R
- R28, R38: value 10R -> 22R/2-3W; device rcl:R-EU_R0805 -> rcl:R-EU_R2512
- R29: value 100R -> 1R
- R3: value ??? -> 120R
- R30: value 22R/2W -> 30K; device rcl:R-EU_R2512 -> rcl:R-EU_R0805
- R31: value 100R -> 10R
- R32: value 22R/2W -> 220K; device rcl:R-EU_R2512 -> rcl:R-EU_R1206
- R33, R41: value 1R -> 10R
- R34: value 30K -> 10R
- R35: value 10R -> 47K
- R36: value 220K -> 1K; device rcl:R-EU_R1206 -> rcl:R-EU_R0805
- R37: value 10R -> 1R
- R39: value 47K -> 22R/2-3W; device rcl:R-EU_R0805 -> rcl:R-EU_R2512
- R40: value 1K -> 100K
- R42: value 22R/2W -> 1K; device rcl:R-EU_R2512 -> rcl:R-EU_R0805
- R43: value 22R/2W -> 6K8; device rcl:R-EU_R2512 -> rcl:R-EU_R0805
- R44: value 100K -> 22R
- R45: value 10R -> 22R
- R47, R53: value 6K8 -> 30K
- R48: value 22R -> 82K
- R49: value 22R -> 1K
- R50: value 1K -> N.C.
- R51: value 30K -> 4K7
- R52: value 82K -> 1K
- R54: value 1K -> 10K
- R55: value 6K8 -> 100R
- R56: device rcl:R-EU_R0805 -> rcl:R-EU_R1210
- R57: value 3K9 -> 22R/2-3W; device rcl:R-EU_R0805 -> rcl:R-EU_R2512
- R58: value 1K -> 22R/2-3W; device rcl:R-EU_R0805 -> rcl:R-EU_R2512
- R59: value 27K -> 3R3
- R61: value 100R -> 47K
- R62: value N.C. -> 3R3; device rcl:R-EU_R1210 -> rcl:R-EU_R0805
- R63, R64: value 22R/3W -> 22R/2-3W
- R65: value 3R3 -> 10K
- R66: value 10R -> 316K
- R67: value 47K -> 10K
- R68: value 3R3 -> 750R
- R69: value 22R/3W -> 750R; device rcl:R-EU_R2512 -> rcl:R-EU_R0805
- R7: value 33K -> 220K; device rcl:R-EU_R1210 -> rcl:R-EU_R1206
- R70: value 22R/3W -> 470R; device rcl:R-EU_R2512 -> rcl:R-EU_R0805
- R71: value 10K -> 12K
- R72: value 316K -> 3K3
- R73: value 10K -> 750R
- R74: value 750R -> 30K
- R75: value 0R -> 10K
- R76: value 750R -> 16K
- R77: value 470R -> 220R
- R8: value 33K -> 100K; device rcl:R-EU_R1210 -> rcl:R-EU_R0805
- R9: value 100K -> 120R
- TP6: device EEZ_Lib1:TEST_POINT-2 -> EEZ_Lib1:PCB_TEST_TABSHIELD
- TP7: device EEZ_Lib1:PCB_TEST_TABSHIELD -> EEZ_Lib1:TEST_POINT-2
- TR1: device EEZ_Lib1:FERYSTER_5572 -> EEZ_inductors_and_transformers:FERYSTER_5572
- X1: value B2B-ZR -> 39-30-1039; device EEZ_Lib1:B2B-ZR -> EEZ_Lib1:MINIFIT_39301039-CREEPAGE
- X2: value 39-30-1039 -> B2B-ZR; device EEZ_Lib1:MINIFIT_39301039-CREEPAGE -> EEZ_Lib1:B2B-ZR
- ZD3: value MMSZ5230BT1G -> MMSZ5V1T1G
Connections:
- removed net +15V: D2.A, R5.1, TR1.S3_DOT
- removed net +15V_REC2: C11.+, C9.2, D2.C, L2.1
- removed net +6V: C22.1, C25.1, D7.C, IC2.IN, L4.2, LED1.A, R23.2, R66.1
- removed net -7V_REC2: C14.-, C19.2, D5.A, L3.1
- removed net -9V: C15.2, C16.2, D6.A, IC1.IN, L3.2, X3-8.S
- removed net AGND: C37.1, C42.2, C45.1, C48.1, C49.1, C50.1, C51.1, C52.2, C53.2, IC4.DISABLE, IC4.GNDI, IC5.AGND, IC5.FB, IC5.PGND, IC6P.V-, JP3.2, OK3.EMIT, Q5.C, Q7.C, R24.2, R25.2, R26.2, R33.1, R33.2, R34.1, R47.2, R51.2, R52.2, R55.2, R58.2, R59.2, R60.2, TR2.S_DOT, ZD4.A, ZD5.A
- removed net AUX_DC: C3.2, C7.+, D1.C, Q1.C, R11.1, R4.1
- removed net FB3: OK1.C, R23.1, ZD3.C
- removed net N$1: C70.2, IC8A.-IN, R75.2, R76.1, R80.1
- removed net N$103: C18.1, JP2.COM
- removed net N$104: C26.1, R22.1
- removed net N$106: D10.C, D11.C, R15.2
- removed net N$107: IC3.BR, R20.1, R9.2
- removed net N$108: R6.2, R9.1
- removed net N$28: C1.1, C2A.2, L1-1.2, R1.1, SAR1.P$1, X2-2.1
- removed net N$30: C1.2, C4A.2, L1-2.2, R2.2, SAR2.P$1, X2-3.1
- removed net N$41: R30.1, R32.2
- removed net N$47: Q7.B, R53.2, R55.1
- removed net N$87: IC2.FB, R14.2, R17.1
- removed net N$89: OK1.A, R16.2
- removed net N$90: LED1.C, R18.1
- removed net N$91: C10.2, D3.C, R8.2
- removed net N$92: C26.2, C27.1, IC3.FB, OK1.COL
- removed net N$95: C28.1, IC3.ZCD, R12.1, R15.1, R21.2
- removed net N$98: C21.1, R13.2
- removed net VIPER_VDD: C20.1, IC3.VDD, R11.2, ZD2.C
- new net +15V_REC: C10.+, D2.C, L2.1, R5.1
- new net -7V_REC: C14.-, D4.A, L3.1, R9.1
- new net 15VAC: C9.2, D2.A, TR1.S3_DOT
- new net AC_L_IN: C1.1, C4A.2, L1-1.2, R1.1, SAR1.P$1, X1-1.1
- new net AC_N_IN: C1.2, C5A.2, L1-2.2, R2.2, SAR2.P$1, X1-2.1
- new net AUX_REC: C7.+, D1.C, Q1.C, R3.1, R4.1
- new net FB2: OK1.C, R19.1, ZD3.C
- new net N$11: LED1.A, R11.2
- new net N$135: OK1.A, R15.2
- new net N$137: C12.2, D3.C, R6.2
- new net N$138: C23.2, C25.1, IC1.FB, OK1.COL
- new net N$141: C24.1, IC1.ZCD, R13.1, R14.1, R16.2
- new net N$144: C16.1, R9.2
- new net N$152: C23.1, R18.1
- new net N$155: D7.C, D8.C, R14.2
- new net N$20: IC1.BR, R17.1, R8.2
- new net N$27: C18.2, C21.+, D6.C, IC1.VDD, ZD2.C
- new net N$4: C17.1, JP2.COM
- net +12V: now also C26.2, C27.2, C49.1, IC4P.V+, R23.2, R34.2, R41.2, X2-1.1; no longer C29.2, C30.2, C52.1, IC6P.V+, R27.2, R38.2, R45.2, X1-1.1
- net +2.5VREF: now also C71.1, IC7-1.+IN1, R67.2, R72.1; no longer C74.1, IC9-1.+IN1, R73.2, R79.1
- net +5VREF: now also C45.2, C50.1, IC3.REF, R33.1, R51.2; no longer C48.2, C53.1, IC5.REF, NTC1.P$1, R37.1, R53.1, R57.2
- net +6V_REC: now also C20.+, D5.C, R10.1, R15.1; no longer C21.2, C24.+, D8.C, R16.1
- net -15V: now also C10.-, C11.2, X3-3.S; no longer C11.-, C12.2, X3-2.S
- net 0V: now also C18.1, C21.-, C24.2, C25.2, C26.1, C27.1, C28.-, C29.-, C33.1, C34.1, C35.2, C36.2, C37.2, C41.2, C42.1, C43.1, C44.1, C45.1, C48.1, C49.2, C50.2, D12.A, D8.A, IC1.GND, IC2.DISABLE, IC2.GNDB, IC2.GNDI, IC3.AGND, IC3.FB, IC3.PGND, IC4P.V-, OK3.EMIT, Q5.C, R16.1, R17.2, R18.2, R21.2, R29.1, R29.2, R30.1, R35.2, R37.1, R37.2, R43.2, R47.2, R48.2, R52.2, R53.2, R54.2, TP1.P$1, TP4.P$1, TR2.S, X2-2.1, ZD4.A, ZD5.A; no longer C20.2, C27.2, C28.2, C29.1, C30.1, C31.-, C32.-, C36.1, C38.2, C43.2, C44.2, D11.A, D15.A, IC3.GND, IC4.GNDB, JP3.1, R21.1, R39.2, R41.1, R41.2, TP3.P$1, X1-2.1
- net 6VAC: now also C19.2, D5.A; no longer D8.A, R13.1
- net 7VAC: now also C16.2, D4.C; no longer D5.C, R10.1
- net AUX_AC: now also C3.2, D6.A, D7.A, R13.2; no longer D10.A, R12.2, R3.1
- net BUCK_OUT: now also C30.2, C31.2, C32.2, D12.C, IC2.GNDA, TP3.P$1; no longer C33.2, C34.2, C35.2, D15.C, IC4.GNDA, TP2.P$1
- net CLAMP_C: now also C43.2, C44.2, D15.C, D16.C, R38.1, R39.1; no longer C46.2, C47.2, D18.C, D19.C, R42.1, R43.1
- net CT_OUT: now also D9.C, R21.1, R22.1, R49.1; no longer D12.C, R25.1, R26.1, R54.1
- net DC_BUS: now also C12.1, C28.+, C29.+, C33.2, R32.1, R38.2, R39.2, TR2.P_DOT; no longer C10.1, C31.+, C32.+, C36.2, R36.1, R42.2, R43.2, TR2.P
- net DC_OUT: now also C11.1, X3-2.S; no longer C12.1, X3-3.S
- net FB: now also R71.1, R75.2, R76.2; no longer C75.2, IC10.REF, R78.1, R82.2, R83.2, R86.2, R87.2, TP7.P$1
- net GND: now also C17.2, C20.-, C51.-, C52.-, C53.-, C54.2, C55.2, C56.2, C59.1, C62.2, C70.-, C71.2, IC5.GND, IC5.VS, IC6A.+IN, IC6B.+IN, IC7-1.VCC-, LED1.C, Q7.S, R61.2, TP2.P$1, TP7.GND; no longer C16.1, C17.1, C18.2, C23.-, C24.-, C25.2, C54.-, C55.-, C56.-, C59.2, C62.1, C67.2, C68.2, C69.2, C73.-, C74.2, D4.C, D9.A, IC1.GND, IC10.A, IC2.GND, IC7.GND, IC7.VS, IC8A.+IN, IC8B.+IN, IC9-1.VCC-, Q9.S, R17.2, R18.2, R67.2, R87.1, TP1.P$1, TP6.GND
- net HD: now also IC3.HD, R25.2; no longer IC5.HD, R29.2
- net HI_OUT: now also D11.A, IC2.VOA, R24.2; no longer D14.A, IC4.VOA, R28.2
- net ISO_FB: now also C46.2, IC3.COMP, R50.1, TP6.P$1; no longer C50.2, IC5.COMP, Q7.E, R56.1, TP5.P$1
- net LD: now also IC3.LD, R27.2; no longer IC5.LD, R31.2
- net LO_OUT: now also D14.A, IC2.VOB, R31.1; no longer D17.A, IC4.VOB, R35.1
- net L_PULL: now also D15.A, L5.P$1, R26.2, TR3.P; no longer C41.2, D18.A, L6.P$1, TR3.P_DOT
- net L_PUSH: now also C38.2, D16.A, L6.P$1, TR3.P_DOT; no longer D19.A, L5.P$1, R30.2, TR3.P
- net N$10: now also C68.2, IC7-1.-IN1, R74.1, R75.1; no longer C71.2, IC9-1.-IN1, R81.1, R82.1
- net N$100: now also R46.1; no longer R50.1
- net N$12: now also R66.1, R71.2; no longer R72.1, R78.2
- net N$126: now also D17.C, D18.C; no longer D20.C, D21.C
- net N$13: now also D19.C, R44.1; no longer D22.C, R48.1
- net N$130: now also D17.A; no longer D20.A
- net N$132: now also IC6B.-IN, R65.2, R67.1; no longer IC8B.-IN, R71.2, R73.1
- net N$134: now also C67.1, IC6A.OUT, R77.2; no longer C70.1, IC8A.OUT, R84.2
- net N$14: now also D20.C, R45.1; no longer D23.C, R49.1
- net N$15: now also B1.AC2; no longer B1.AC1
- net N$16: now also R36.2; no longer R40.2
- net N$17: now also C38.1, R28.1; no longer C76.2, R86.1
- net N$18: now also IC5.MOT, R61.1; no longer IC7.MOT, R67.1
- net N$19: now also IC3.RT/SYNC, R48.1; no longer IC5.RT/SYNC, R52.1
- net N$2: now also R32.2, R40.1; no longer R36.2, R44.1
- net N$21: now also D11.C, R24.1; no longer D14.C, R28.1
- net N$22: now also IC3.TIME, R47.1; no longer IC5.TIME, R51.1
- net N$23: now also C42.2, IC3.SS; no longer C45.2, IC5.SS
- net N$24: now also B1.AC1; no longer B1.AC2
- net N$25: now also IC3.UVLO, R42.1; no longer IC5.UVLO, R46.1
- net N$26: now also IC4B.-IN, R51.1, R53.1; no longer IC6B.-IN, R57.1, R59.1
- net N$29: now also D14.C, R31.2, R35.1; no longer D17.C, R35.2, R39.1
- net N$3: now also C30.1, C31.1, C32.1, D10.C, IC2.VDDA; no longer C33.1, C34.1, C35.1, D13.C, IC4.VDDA
- net N$31: now also D10.A, R23.1; no longer D13.A, R27.1
- net N$32: now also R36.1; no longer R40.1
- net N$35: now also C48.2, R50.2; no longer C51.2, R56.2
- net N$36: now also IC2.VIA, R25.1; no longer IC4.VIA, R29.1
- net N$37: now also C47.2, IC3.CS, R49.2; no longer C49.2, IC5.CS, R54.2
- net N$38: now also IC4B.OUT, R46.2, R52.1; no longer IC6B.OUT, R50.2, R58.1
- net N$40: now also IC2.VIB, R27.1; no longer IC4.VIB, R31.1
- net N$42: now also IC4A.-IN, IC4A.OUT, IC4B.+IN; no longer IC6A.-IN, IC6A.OUT, IC6B.+IN
- net N$48: now also IC2.DT, R30.2; no longer IC4.DT, R34.2
- net N$5: now also R26.1, R28.2; no longer C41.1, R32.1
- net N$50: now also D9.A, R20.1, TR2.S_DOT; no longer D12.A, R24.1, TR2.S
- net N$53: now also IC6B.OUT, R65.1, R69.2; no longer IC8B.OUT, R71.1, R76.2
- net N$54: now also C40.1, C41.1, IC3.VCC, IC3.VIN, R41.1; no longer C43.1, C44.1, IC5.VCC, IC5.VIN, R45.1
- net N$55: now also C35.1, C36.1, C37.1, D13.C, IC2.VDDB; no longer C38.1, C39.1, C40.1, D16.C, IC4.VDDB
- net N$56: now also TR2.P; no longer TR2.P_DOT
- net N$57: now also IC7-2.+IN, JP3.COM; no longer IC9-2.+IN, JP4.COM
- net N$58: now also JP3.NO; no longer JP4.NO
- net N$6: now also C61.1, C62.1, IC5.VCC, R60.2; no longer C64.1, C65.1, IC7.VCC, R66.2
- net N$63: now also D13.A, R34.1; no longer D16.A, R38.1
- net N$64: now also C67.2, IC6A.-IN, R68.2, R69.1, R73.1; no longer R74.2, R75.1
- net N$66: now also C60.1, R57.2, R58.2; no longer C63.1, R63.2, R64.2
- net N$67: now also C64.1, R63.2, R64.2; no longer C67.1, R69.2, R70.2
- net N$7: now also IC4A.+IN, R54.1; no longer IC6A.+IN, NTC1.P$2, R60.1
- net N$74: now also D21.C, IC5.GATE1, R59.2; no longer D24.C, IC7.GATE1, R65.2
- net N$75: now also D22.C, IC5.GATE2, R62.2; no longer D25.C, IC7.GATE2, R68.2
- net N$76: now also C68.1, C69.1, IC7-1.OUT1; no longer C71.1, C72.1, C75.1, C76.1, IC10.C, IC9-1.OUT1, R85.2
- net N$8: now also C59.2, R56.1; no longer C62.2, R62.1
- net N$9: now also C69.2, R74.2; no longer C72.2, R81.2
- net NFB_OFFSET: now also C70.+, R68.1, R76.1, R77.1; no longer C73.+, R74.1, R83.1, R84.1
- net OK_A: now also R70.1; no longer R77.1, R85.1
- net PE: now also C5A.1, X1-3.1, X3-8.S; no longer C2A.1, X2-1.1
- net POUT+: now also C51.+, C52.+, C53.+, C54.1, R55.1, R66.2; no longer C54.+, C55.+, C56.+, C57.1, R61.1, R72.2
- net PREG_OUT+: now also C55.1, C56.1, C57.1, R55.2, R56.2, TP7.TIP; no longer C59.1, C60.1, C61.1, R61.2, R62.2, TP6.TIP
- net PULL: now also D20.A, IC3.PULL, R45.2; no longer D23.A, IC5.PULL, R49.2
- net PUSH: now also D19.A, IC3.PUSH, R44.2; no longer D22.A, IC5.PUSH, R48.2
- net PWRGOOD: now also R12.2; no longer IC2.!ERROR, R19.2
- net REF: now also C34.2, IC2.VDDI, R33.2; no longer C37.2, IC4.VDDI, R37.2
- net S1_DOT_OUT: now also IC5.VD1, Q7.D, R57.1, R58.1; no longer IC7.VD1, Q8.D, R63.1, R64.1
- net S2_OUT: now also IC5.VD2, Q8.D, R63.1, R64.1; no longer IC7.VD2, Q9.D, R69.1, R70.1
- net SR_OUT1: now also D21.A, Q7.G, R59.1; no longer D24.A, Q8.G, R65.1
- net SR_OUT2: now also D22.A, Q8.G, R62.1; no longer D25.A, Q9.G, R68.1
- net ULVO: now also C39.1, D18.A, R40.2, R42.2, R43.1, TP5.P$1; no longer C42.1, D21.A, R44.2, R46.2, R47.1, TP4.P$1
- net U_MON: now also JP3.NC; no longer JP4.NC
- net U_MON1: now also IC7-2.-IN, IC7-2.OUT, R73.2; no longer IC9-2.-IN, IC9-2.OUT, R80.2
- net V+: now also C22.1, C63.1, IC6P.V+, IC7-1.VCC+, L4.2, R11.1, R12.1, R19.2, R60.1, R70.2, R72.2; no longer C23.+, C69.1, D7.A, D9.C, IC2.OUT, IC8P.V+, IC9-1.VCC+, R14.1, R19.1, R77.2, R79.2
- net V-: now also C15.2, C65.1, IC6P.V-, L3.2; no longer C17.2, C68.1, D4.A, D6.C, IC1.OUT, IC8P.V-
- net VIPER_D: now also IC1.DRAIN; no longer IC3.DRAIN
Other:
- note added: ""Power" (yellow)"
- note added: "Cfb"
- note added: "Cfb1"
- note added: "Rfb1"
- note removed: "18p"
- note removed: "5R1 (4R7)"
- note removed: "LM5041B Vcc"
- note removed: "N.C."
- note removed: "Optional NFB if tracker is not used!"
- note removed: "Post-regulator pass mosfet Drain"
- note removed: "Post-regulator pass mosfet Vbias"
- note removed: "US1K-DIO"
- note removed: "V+ for sync rectifier gate driver"
- note removed: "V- for downprogrammer"
- moved on the sheet: B1, C1, C12, C13, C14, C15, C16, C17, C18, C19, C2, C22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

Commit message: PWRGOOD renamed to FAULT
Connections:
- net PWRGOOD renamed !FAULT
Other:
- note added: "!FAULT! 4"
- note added: "Bias+ 2"
- note added: "Bias- 3"
- note added: "PE 8"
- note added: "V+ 5"
- note added: "V- 7"
- note removed: "+5 Vdc 5"
- note removed: "-5 Vdc 7"
- note removed: "-9 Vdc 8"
- note removed: "Bias+ 3"
- note removed: "Bias- 2"
- note removed: "PWRGOOD 4"
Changed lines of the file:
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@@
 <circle x="242.57" y="146.05" radius="0.635" width="0.1524" layer="101"/>
 <text x="240.665" y="146.685" size="1.4224" layer="101" rot="R180">U_MON 1</text>
-<text x="240.665" y="144.145" size="1.4224" layer="101" rot="R180">Bias- 2</text>
+<text x="240.665" y="144.145" size="1.4224" layer="101" rot="R180">Bias+ 2</text>
 <wire x1="243.84" y1="127" x2="241.3" y2="127" width="0.1524" layer="101"/>
 <wire x1="241.3" y1="127" x2="241.3" y2="147.32" width="0.1524" layer="101"/>
@@
 <wire x1="243.84" y1="147.32" x2="243.84" y2="127" width="0.1524" layer="101"/>
 <circle x="242.57" y="140.97" radius="0.635" width="0.1524" layer="101"/>
-<text x="240.665" y="141.605" size="1.4224" layer="101" rot="R180">Bias+ 3</text>
+<text x="240.665" y="141.605" size="1.4224" layer="101" rot="R180">Bias- 3</text>
 <circle x="242.57" y="138.43" radius="0.635" width="0.1524" layer="101"/>
-<text x="240.665" y="139.065" size="1.4224" layer="101" rot="R180">PWRGOOD 4</text>
+<text x="240.665" y="139.065" size="1.4224" layer="101" rot="R180">!FAULT! 4</text>
 <circle x="242.57" y="135.89" radius="0.635" width="0.1524" layer="101"/>
-<text x="240.665" y="136.525" size="1.4224" layer="101" rot="R180">+5 Vdc 5</text>
+<text x="240.665" y="136.525" size="1.4224" layer="101" rot="R180">V+ 5</text>
 <circle x="242.57" y="133.35" radius="0.635" width="0.1524" layer="101"/>
 <text x="240.665" y="133.985" size="1.4224" layer="101" rot="R180">GND 6</text>
 <circle x="242.57" y="130.81" radius="0.635" width="0.1524" layer="101"/>
-<text x="240.665" y="131.445" size="1.4224" layer="101" rot="R180">-5 Vdc 7</text>
+<text x="240.665" y="131.445" size="1.4224" layer="101" rot="R180">V- 7</text>
 <circle x="242.57" y="128.27" radius="0.635" width="0.1524" layer="101"/>
-<text x="240.665" y="128.905" size="1.4224" layer="101" rot="R180">-9 Vdc 8</text>
+<text x="240.665" y="128.905" size="1.4224" layer="101" rot="R180">PE 8</text>
 <text x="224.155" y="149.225" size="1.778" layer="101">X3 8-pin output connector</text>
 <circle x="242.57" y="161.29" radius="0.635" width="0.1524" layer="101"/>
@@
 <text x="226.695" y="167.005" size="1.778" layer="101">X2 3-pin input connector</text>
 <text x="156.718" y="40.64" size="1.27" layer="103">"Power" (yellow)</text>
+<rectangle x1="184.785" y1="55.88" x2="190.5" y2="64.77" layer="97"/>
 </plain>
 <instances>
@@
 </instance>
 <instance part="LED1" gate="G$1" x="162.56" y="48.26" smashed="yes">
-<attribute name="NAME" x="162.306" y="51.308" size="1.778" layer="95" rot="R90"/>
-<attribute name="VALUE" x="165.1" y="51.308" size="1.27" layer="96" rot="R90"/>
+<attribute name="NAME" x="164.973" y="49.784" size="1.778" layer="95"/>
+<attribute name="VALUE" x="164.973" y="47.625" size="1.27" layer="96"/>
 </instance>
 <instance part="R11" gate="G$1" x="162.56" y="63.5" smashed="yes" rot="MR270">
@@
 </segment>
 </net>
-<net name="PWRGOOD" class="0">
+<net name="!FAULT" class="0">
 <segment>
 <pinref part="R12" gate="G$1" pin="2"/>
@@
 <junction x="193.04" y="45.72"/>
 <wire x1="193.04" y1="50.8" x2="195.58" y2="50.8" width="0.1524" layer="91"/>
-<label x="211.455" y="50.8" size="1.27" layer="102" rot="R180" xref="yes"/>
+<label x="207.645" y="50.8" size="1.27" layer="102" rot="R180" xref="yes"/>
 </segment>
 </net>
@@
 </segment>
 </net>
-<net name="PWRGOOD" class="0">
+<net name="!FAULT" class="0">
 <segment>
 <pinref part="OK2" gate="G$1" pin="COL"/>

Commit message: #1, power inductors rotated, shorter PUSH gate trace
Parts:
- removed TP7: (no value), EEZ_Lib1:TEST_POINT-2
- TP6: device EEZ_Lib1:PCB_TEST_TABSHIELD -> EEZ_Lib1:TEST_POINT-2
Connections:
- net GND: now also TP6.GND; no longer TP7.GND
- net ISO_FB: now also TP5.P$1; no longer TP6.P$1
- net PREG_OUT+: now also TP6.TIP; no longer TP7.TIP
- net ULVO: no longer TP5.P$1
Other:
- moved on the sheet: TP5
Changed lines of the file:
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@@
 <setting verticaltext="up"/>
 </settings>
-<grid distance="0.025" unitdist="inch" unit="inch" style="lines" multiple="4" display="no" altdistance="0.01" altunitdist="inch" altunit="inch"/>
+<grid distance="0.1" unitdist="inch" unit="inch" style="lines" multiple="1" display="no" altdistance="0.01" altunitdist="inch" altunit="inch"/>
 <layers>
 <layer number="1" name="Top" color="4" fill="1" visible="no" active="no"/>
@@
 <part name="R28" library="rcl" deviceset="R-EU_" device="R2512" value="22R/2-3W"/>
 <part name="C44" library="rcl" deviceset="C-EU" device="C1812" value="100n/500V"/>
-<part name="TP7" library="EEZ_Lib1" deviceset="TEST_POINT" device="-2"/>
+<part name="TP6" library="EEZ_Lib1" deviceset="TEST_POINT" device="-2"/>
 <part name="D21" library="diode" deviceset="DIODE-" device="SOD323-W" value="1N5819HW-7-F"/>
 <part name="D22" library="diode" deviceset="DIODE-" device="SOD323-W" value="1N5819HW-7-F"/>
@@
 <part name="TP4" library="EEZ_Lib1" deviceset="PCB_TEST_TAB" device="SHIELD"/>
 <part name="TP3" library="EEZ_Lib1" deviceset="PCB_TEST_TAB" device="SHIELD"/>
-<part name="TP5" library="EEZ_Lib1" deviceset="PCB_TEST_TAB" device="SHIELD"/>
 <part name="SUPPLY10" library="supply2" deviceset="V-" device=""/>
 <part name="P+1" library="supply2" deviceset="V+" device=""/>
 <part name="ZD6" library="EEZ_Lib1" deviceset="PSMAXX" device="" value="SMAJ58A-TR"/>
-<part name="TP6" library="EEZ_Lib1" deviceset="PCB_TEST_TAB" device="SHIELD"/>
+<part name="TP5" library="EEZ_Lib1" deviceset="PCB_TEST_TAB" device="SHIELD"/>
 <part name="X2" library="EEZ_Lib1" deviceset="B2B-ZR" device=""/>
 <part name="C58" library="rcl" deviceset="C-EU" device="C0805" value="100n/100V"/>
@@
 <rectangle x1="213.36" y1="106.045" x2="217.805" y2="112.395" layer="97"/>
 <rectangle x1="216.535" y1="162.56" x2="220.98" y2="170.815" layer="97"/>
-<text x="167.64" y="55.88" size="1.27" layer="100">Route traces between PP MOSFETs and transformer primary as short as possible and of equal length</text>
+<text x="165.1" y="55.88" size="1.27" layer="100">Route traces between PP MOSFETs and transformer primary as short as possible and of equal length</text>
 <text x="6.858" y="99.06" size="1.27" layer="103">"Fault" (red)</text>
 <wire x1="27.94" y1="147.32" x2="27.94" y2="35.56" width="0.1524" layer="97" style="shortdash"/>
@@
 <attribute name="VALUE" x="193.04" y="154.94" size="1.778" layer="96" rot="R90"/>
 </instance>
-<instance part="TP5" gate="G$1" x="38.1" y="96.52" smashed="yes" rot="R90">
-<attribute name="NAME" x="35.56" y="98.425" size="1.778" layer="95"/>
-<attribute name="VALUE" x="40.64" y="96.52" size="1.778" layer="96" rot="R90"/>
-</instance>
-<instance part="TP6" gate="G$1" x="38.1" y="60.96" smashed="yes" rot="R90">
+<instance part="TP5" gate="G$1" x="38.1" y="60.96" smashed="yes" rot="R90">
 <attribute name="NAME" x="35.56" y="62.865" size="1.778" layer="95"/>
 <attribute name="VALUE" x="40.64" y="60.96" size="1.778" layer="96" rot="R90"/>
@@
 <junction x="43.18" y="93.98"/>
 <wire x1="43.18" y1="93.98" x2="38.1" y2="93.98" width="0.1524" layer="91"/>
-<pinref part="TP5" gate="G$1" pin="P$1"/>
 <junction x="38.1" y="93.98"/>
 <pinref part="D18" gate="G$1" pin="A"/>
@@
 <wire x1="38.1" y1="58.42" x2="63.5" y2="58.42" width="0.1524" layer="91"/>
 <wire x1="71.12" y1="58.42" x2="63.5" y2="58.42" width="0.1524" layer="91"/>
-<pinref part="TP6" gate="G$1" pin="P$1"/>
+<pinref part="TP5" gate="G$1" pin="P$1"/>
 <junction x="38.1" y="58.42"/>
 </segment>
@@
 <segment>
 <pinref part="Q6" gate="G$1" pin="S"/>
-<wire x1="208.28" y1="66.04" x2="162.56" y2="66.04" width="0.1524" layer="91"/>
-<wire x1="162.56" y1="66.04" x2="162.56" y2="101.6" width="0.1524" layer="91"/>
-<wire x1="162.56" y1="101.6" x2="152.4" y2="109.22" width="0.1524" layer="91"/>
 <junction x="152.4" y="109.22"/>
 <pinref part="Q4" gate="G$1" pin="S"/>
-<wire x1="233.68" y1="83.82" x2="233.68" y2="63.5" width="0.1524" layer="91"/>
-<wire x1="233.68" y1="63.5" x2="160.02" y2="63.5" width="0.1524" layer="91"/>
-<wire x1="160.02" y1="63.5" x2="160.02" y2="101.6" width="0.1524" layer="91"/>
-<wire x1="160.02" y1="101.6" x2="152.4" y2="109.22" width="0.1524" layer="91"/>
-<wire x1="157.48" y1="43.18" x2="157.48" y2="101.6" width="0.1524" layer="91"/>
+<wire x1="233.68" y1="83.82" x2="233.68" y2="68.58" width="0.1524" layer="91"/>
+<wire x1="218.44" y1="63.5" x2="157.48" y2="63.5" width="0.1524" layer="91"/>
+<wire x1="157.48" y1="63.5" x2="157.48" y2="101.6" width="0.1524" layer="91"/>
 <wire x1="157.48" y1="101.6" x2="152.4" y2="109.22" width="0.1524" layer="91"/>
 <pinref part="C41" gate="G$1" pin="2"/>
@@
 <wire x1="116.84" y1="132.08" x2="119.38" y2="132.08" width="0.1524" layer="91"/>
 <junction x="119.38" y="132.08"/>
-<wire x1="208.28" y1="73.66" x2="208.28" y2="66.04" width="0.1524" layer="91"/>
+<wire x1="208.28" y1="73.66" x2="208.28" y2="68.58" width="0.1524" layer="91"/>
 <wire x1="182.88" y1="137.16" x2="177.8" y2="137.16" width="0.1524" layer="91"/>
 <pinref part="SH1" gate="SH" pin="GND_B"/>
@@
 <pinref part="C43" gate="G$1" pin="1"/>
 <pinref part="C44" gate="G$1" pin="1"/>
-<wire x1="218.44" y1="76.2" x2="210.82" y2="76.2" width="0.1524" layer="91"/>
-<wire x1="210.82" y1="76.2" x2="208.28" y2="73.66" width="0.1524" layer="91"/>
-<junction x="208.28" y="73.66"/>
-<wire x1="223.52" y1="76.2" x2="231.14" y2="76.2" width="0.1524" layer="91"/>
-<wire x1="231.14" y1="76.2" x2="233.68" y2="83.82" width="0.1524" layer="91"/>
-<junction x="233.68" y="83.82"/>
 <pinref part="C29" gate="G$1" pin="-"/>
 <pinref part="C28" gate="G$1" pin="-"/>
@@
 <junction x="134.62" y="5.08"/>
 <pinref part="IC4" gate="P" pin="V-"/>
-<wire x1="157.48" y1="43.18" x2="114.3" y2="43.18" width="0.1524" layer="91"/>
 <junction x="114.3" y="43.18"/>
+<wire x1="218.44" y1="76.2" x2="218.44" y2="71.12" width="0.1524" layer="91"/>
+<junction x="220.98" y="68.58"/>
+<wire x1="223.52" y1="76.2" x2="223.52" y2="71.12" width="0.1524" layer="91"/>
+<wire x1="223.52" y1="71.12" x2="220.98" y2="68.58" width="0.1524" layer="91"/>
+<junction x="220.98" y="68.58"/>
+<wire x1="220.98" y1="68.58" x2="218.44" y2="71.12" width="0.1524" layer="91"/>
+<wire x1="208.28" y1="68.58" x2="220.98" y2="68.58" width="0.1524" layer="91"/>
+<wire x1="233.68" y1="68.58" x2="220.98" y2="68.58" width="0.1524" layer="91"/>
+<junction x="220.98" y="68.58"/>
+<wire x1="114.3" y1="43.18" x2="157.48" y2="43.18" width="0.1524" layer="91"/>
+<wire x1="157.48" y1="43.18" x2="157.48" y2="60.96" width="0.1524" layer="91"/>
+<wire x1="157.48" y1="60.96" x2="220.98" y2="60.96" width="0.1524" layer="91"/>
+<wire x1="220.98" y1="60.96" x2="220.98" y2="68.58" width="0.1524" layer="91"/>
+<wire x1="220.98" y1="68.58" x2="218.44" y2="66.04" width="0.1524" layer="91"/>
+<wire x1="218.44" y1="66.04" x2="218.44" y2="63.5" width="0.1524" layer="91"/>
 </segment>
 <segment>
@@
 <pinref part="R44" gate="G$1" pin="2"/>
 <wire x1="182.88" y1="86.36" x2="182.88" y2="93.98" width="0.1524" layer="91"/>
-<wire x1="154.94" y1="86.36" x2="182.88" y2="86.36" width="0.1524" layer="91"/>
+<wire x1="172.72" y1="86.36" x2="182.88" y2="86.36" width="0.1524" layer="91"/>
 <junction x="182.88" y="86.36"/>
 <label x="176.53" y="86.995" size="1.27" layer="102"/>
 <pinref part="IC3" gate="A" pin="PUSH"/>
-<wire x1="101.6" y1="71.12" x2="154.94" y2="71.12" width="0.1524" layer="91"/>
-<wire x1="154.94" y1="71.12" x2="154.94" y2="86.36" width="0.1524" layer="91"/>
+<wire x1="101.6" y1="71.12" x2="172.72" y2="71.12" width="0.1524" layer="91"/>
+<wire x1="172.72" y1="71.12" x2="172.72" y2="86.36" width="0.1524" layer="91"/>
 </segment>
 </net>
@@
 <attribute name="VALUE" x="163.195" y="61.595" size="1.778" layer="96"/>
 </instance>
-<instance part="TP7" gate="G$1" x="233.68" y="152.4" smashed="yes">
+<instance part="TP6" gate="G$1" x="233.68" y="152.4" smashed="yes">
 <attribute name="NAME" x="231.775" y="155.575" size="1.778" layer="95"/>
 <attribute name="VALUE" x="236.855" y="150.495" size="1.778" layer="96"/>
@@
 <pinref part="SUPPLY12" gate="GND" pin="GND"/>
 <wire x1="246.38" y1="139.7" x2="241.3" y2="139.7" width="0.1524" layer="91"/>
-<pinref part="TP7" gate="G$1" pin="GND"/>
+<pinref part="TP6" gate="G$1" pin="GND"/>
 <wire x1="241.3" y1="139.7" x2="233.68" y2="139.7" width="0.1524" layer="91"/>
 <wire x1="233.68" y1="147.32" x2="233.68" y2="139.7" width="0.1524" layer="91"/>
@@
 <wire x1="246.38" y1="160.02" x2="241.3" y2="160.02" width="0.1524" layer="91"/>
 <label x="246.38" y="160.655" size="1.27" layer="102" rot="MR0"/>
-<pinref part="TP7" gate="G$1" pin="TIP"/>
+<pinref part="TP6" gate="G$1" pin="TIP"/>
 <wire x1="241.3" y1="160.02" x2="228.6" y2="160.02" width="0.1524" layer="91"/>
 <wire x1="228.6" y1="152.4" x2="228.6" y2="160.02" width="0.1524" layer="91"/>
