File: Eagle files/EEZ CF-DIC r5B1.brd (EAGLE design)
At the start: 155 x 90 mm, 249 parts, among them IC1 VIPer35L, IC2 SI8233BB-D-IS1, IC3 LM5041B, IC4 LM258D, IC5 IR11688STRPBF, IC6 TL072, IC7 TL103W, IC8 TL431, P1 T910W-50K, Q1 MMBT5551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

Commit message: X2 rotated for easier cable insertion
Parts:
- X2: device con-molex:70543-08 -> EEZ_connectors:70543-08
- moved JP2 0.71 mm to (145.3, 29.9)
- moved X2 0.51 mm to (150.4, 18.2), turned to 90 degrees
Connections:
- net -15V: now also X2.6; no longer X2.3
- net DC_OUT: now also X2.7; no longer X2.2
- net GND: now also X2.3; no longer X2.6
- net N$1: now also X2.5; no longer X2.4
- net PE: now also X2.1; no longer X2.8
- net U_MON: now also X2.8; no longer X2.1
- net V+: now also X2.4; no longer X2.5
- net V-: now also X2.2; no longer X2.7
Routing:
- net GND: track 102.3 -> 101.2 mm
- net -15V: track 45.1 -> 45.6 mm
- net U_MON: track 70.8 -> 71.3 mm
- net V-: track 113.9 -> 113.4 mm
- net V+: track 133.6 -> 133.1 mm
- net N$1: track 44.2 -> 43.7 mm
- net DC_OUT: track 16.5 -> 16.0 mm
Other:
- board text added: "1 PE"
- board text added: "2 V-"
- board text added: "3 Gnd"
- board text added: "4 V+"
- board text added: "5 !FAULT!"
- board text added: "6 Bias-"
- board text added: "7 Bias+"
- board text added: "8 U_MON"
- board text removed: "1 U_MON"
- board text removed: "2 Bias+"
- board text removed: "3 Bias-"
- board text removed: "4 !FAULT!"
- board text removed: "5 V+"
- board text removed: "6 Gnd"
- board text removed: "7 V-"
- board text removed: "8 PE"
