File: Eagle files/EEZ CF-DIC r5B1.sch (EAGLE design)
At the start: 231 parts, among them IC1 VIPer35L, IC2 SI8233BB-D-IS1, IC3 LM5041B, IC4 LM258D, IC5 IR11688STRPBF, IC6 TL072, IC7 TL103W, P1 T910W-50K, Q1 MMBT5551, Q2 C3M0280090D, Q3 C3M0280090D, Q4 C3M0280090D, Q5 NYC0102BLT1G, Q6 C3M0280090D, Q7 IRFS4321PBF, Q8 IRFS4321PBF, X1 39-30-1039, X2 B2B-ZR, X3 90136-1208, X4 B2B-ZR, X5 39-28-1023

Commit message: r5B1 without updated BOM
Parts:
- removed LED1: LTST-C170YKT, EEZ_Lib1:LED0805
- removed LED2: LTST-C170KRKT, EEZ_Lib1:LED0805
- removed TP3, TP4, TP5: (no value), EEZ_Lib1:PCB_TEST_TABSHIELD
- removed TP6: (no value), EEZ_Lib1:TEST_POINT-2
- removed X5: 39-28-1023, EEZ_Lib1:MINIFIT_5566-02A
- removed ZD6: SMAJ58A-TR, EEZ_Lib1:PSMAXX
- added C72, C73: N.C., rcl:C-EUC0805
- added C74: 1n, rcl:C-EUC0805
- added D23: 1N5819HW-7-F, diode:DIODE-SOD323-W
- added D24: BAS316, EEZ_Lib1:DIODESOD323R
- added FAULT: LTST-C170KRKT, EEZ_Lib1:LED0805
- added IC8: TL431, EEZ_Lib1:TL431
- added JP4, JP5, JP6, JP8: JP2-NOCUT, EEZ_Lib1:JP2-NOCUT
- added JP7: JP3-CUT, EEZ_Lib1:JP3-CUT
- added PWR: LTST-C170YKT, EEZ_Lib1:LED0805
- added R78: 12K, rcl:R-EU_R0805
- added R79: 470R, rcl:R-EU_R0805
- added R80, R84: 750R, rcl:R-EU_R0805
- added R81: 10K, rcl:R-EU_R0805
- added R82: 16K, rcl:R-EU_R0805
- added R83: 220R, rcl:R-EU_R0805
- added R85: 6K8, rcl:R-EU_R0805
- added R86: 7K5, rcl:R-EU_R0805
- C15, C22: device rcl:C-EUC1206 -> rcl:C-EUC1210
- C20: device EEZ_Lib1:ECAP5G_10.5MM -> EEZ_Lib1:ECAP5G_13MM
- C28: value UCY2G121MHD -> 10n; device EEZ_Lib1:ECAP7.5G_18MM -> rcl:C-EUC0603
- C29: value UCY2G121MHD -> 100n; device EEZ_Lib1:ECAP7.5G_18MM -> rcl:C-EUC0603
- C30: value 10n -> 100n
- C31, C32: value 100n -> UCY2G121MHD; device rcl:C-EUC0603 -> EEZ_Lib1:ECAP7.5G_18MM
- C38: value 2n2/1kV -> 4n7/200V
- C39: value 10n -> 100n/500V; device rcl:C-EUC0603 -> rcl:C-EUC1812
- C40: value 1u -> 10n
- C41: value 100n -> 1u; device rcl:C-EUC0603 -> rcl:C-EUC0805
- C42: value 1u -> 100n; device rcl:C-EUC0805 -> rcl:C-EUC0603
- C43: value 100n/500V -> 10n; device rcl:C-EUC1812 -> rcl:C-EUC0805
- C44: value 100n/500V -> 100n; device rcl:C-EUC1812 -> rcl:C-EUC0603
- C45: value 100n -> 1n; device rcl:C-EUC0603 -> rcl:C-EUC0805
- C46: value 470p -> 100p
- C47: value 220p -> 100n; device rcl:C-EUC0805 -> rcl:C-EUC0603
- C48: value N.C. -> 1u
- C49: value 100n -> UPW1J152MHD; device rcl:C-EUC0603 -> EEZ_Lib1:ECAP7.5G_18MM
- C50: value N.C. -> UPW1J152MHD; device rcl:C-EUC0603 -> EEZ_Lib1:ECAP7.5G_18MM
- C52: value UPW1J152MHD -> 1u/100V; device EEZ_Lib1:ECAP7.5G_18MM -> rcl:C-EUC1206
- C53: value UPW1J152MHD -> HHXC630ARA330MHA0G; device EEZ_Lib1:ECAP7.5G_18MM -> Panasonic-EEEFK_EEEFP:EEE-FK1J470P-CASE-F; MPN (none) -> EEE-FK1J470P; OC_FARNELL (none) -> 9696032; OC_NEWARK (none) -> 96K9403; PACKAGE (none) -> CASE-F; SUPPLIER (none) -> PANASONIC; TOLERANCE (none) -> ±20 %; VALUE (none) -> 47UF; VOLTAGERATING (none) -> 63 V
- C54: value 1u/100V -> HHXC630ARA330MHA0G; device rcl:C-EUC1206 -> Panasonic-EEEFK_EEEFP:EEE-FK1J470P-CASE-F
- C55: value HHXC630ARA330MHA0G -> 1u/100V; device Panasonic-EEEFK_EEEFP:EEE-FK1J470P-CASE-F -> rcl:C-EUC1206; MPN EEE-FK1J470P -> (none); OC_FARNELL 9696032 -> (none); OC_NEWARK 96K9403 -> (none); PACKAGE CASE-F -> (none); SUPPLIER PANASONIC -> (none); TOLERANCE ±20 % -> (none); VALUE 47UF -> (none); VOLTAGERATING 63 V -> (none)
- C56: value HHXC630ARA330MHA0G -> 100n/100V; device Panasonic-EEEFK_EEEFP:EEE-FK1J470P-CASE-F -> rcl:C-EUC1206
- C57: value 1u/100V -> N.C.
- C58: value 100n/100V -> 4n7/200V; device rcl:C-EUC0805 -> rcl:C-EUC1206
- C60: value 4n7/200V -> N.C.
- C63: value 100n -> 4n7/200V; device rcl:C-EUC0603 -> rcl:C-EUC1206
- C64: value 4n7/200V -> 100n; device rcl:C-EUC1206 -> rcl:C-EUC0603
- C66: value 100n -> 100p; device rcl:C-EUC0603 -> rcl:C-EUC0805
- C67: value 100p -> 100n; device rcl:C-EUC0805 -> rcl:C-EUC0603
- D12: value C3D03060A -> C3D06065A
- D15: value C3D02065E -> US1M-DIO; device EEZ_Lib1:SCHOTTKY-SIC -> EEZ_Lib1:DIODEDO214AA
- D19: value 1N5819HW-7-F -> C3D02065E; device diode:DIODE-SOD323-W -> EEZ_Lib1:SCHOTTKY-SIC
- JP1: value JP3-CUT -> JP2-NOCUT; device EEZ_Lib1:JP3-CUT -> EEZ_Lib1:JP2-NOCUT
- Q2, Q3, Q6: device EEZ_Lib1:N-MOSFETTO247 -> EEZ_Lib1:IRFP240
- Q4: value C3M0280090D -> NYC0102BLT1G; device EEZ_Lib1:N-MOSFETTO247 -> EEZ_Lib1:NYC0102BLT1G
- Q5: value NYC0102BLT1G -> C3M0280090D; device EEZ_Lib1:NYC0102BLT1G -> EEZ_Lib1:IRFP240
- R11: value 470R -> N.C.
- R12, R65: value 10K -> 47K
- R13: value N.C. -> 750R
- R14: value 47K -> 12K
- R15: value 750R -> 1K8
- R16: value 12K -> 47K
- R17: value 1K8 -> 1K
- R18: value 47K -> 10R
- R19: value 1K -> 10K
- R20: value 10K -> 6R2
- R21: value 6R2 -> N.C.
- R22: value N.C. -> 10R
- R23, R24: value 10R -> 100R
- R25: value 100R -> 22R/2-3W; device rcl:R-EU_R0805 -> rcl:R-EU_R2512
- R27: value 100R -> 1R
- R28: value 22R/2-3W -> 30K; device rcl:R-EU_R2512 -> rcl:R-EU_R0805
- R29: value 1R -> 10R
- R30: value 30K -> 220K; device rcl:R-EU_R0805 -> rcl:R-EU_R1206
- R32: value 220K -> 47K; device rcl:R-EU_R1206 -> rcl:R-EU_R0805
- R33: value 10R -> 1K
- R34: value 10R -> 1R
- R35, R61: value 47K -> 22R/2-3W; device rcl:R-EU_R0805 -> rcl:R-EU_R2512
- R36, R42: value 1K -> 100K
- R37: value 1R -> 22R/2-3W; device rcl:R-EU_R0805 -> rcl:R-EU_R2512
- R38, R64: value 22R/2-3W -> 10R; device rcl:R-EU_R2512 -> rcl:R-EU_R0805
- R39, R58: value 22R/2-3W -> 1K; device rcl:R-EU_R2512 -> rcl:R-EU_R0805
- R40: value 100K -> 10R
- R41: value 10R -> 30K
- R43: value 6K8 -> 10K
- R45: value 22R -> 4K7
- R46: value 1K -> 33K
- R47: value 30K -> 51K
- R48: value 82K -> 22R
- R51: value 4K7 -> 750R
- R52: value 1K -> 4K7
- R53: value 30K -> 5K6
- R54: value 10K -> 30K
- R55: value 100R -> 1K
- R56: value N.C. -> 30K; device rcl:R-EU_R1210 -> rcl:R-EU_R0805
- R57: value 22R/2-3W -> 10K; device rcl:R-EU_R2512 -> rcl:R-EU_R0805
- R59: value 3R3 -> 120R
- R60: value 10R -> N.C.; device rcl:R-EU_R0805 -> rcl:R-EU_R1210
- R62: value 3R3 -> 22R/2-3W; device rcl:R-EU_R0805 -> rcl:R-EU_R2512
- R63: value 22R/2-3W -> 3R3; device rcl:R-EU_R2512 -> rcl:R-EU_R0805
- R66: value 316K -> 3R3
- R67: value 10K -> 22R/2-3W; device rcl:R-EU_R0805 -> rcl:R-EU_R2512
- R68: value 750R -> 22R/2-3W; device rcl:R-EU_R0805 -> rcl:R-EU_R2512
- R69: value 750R -> 470R
- R71: value 12K -> 10K
- R72: value 3K3 -> 316K
- R73: value 750R -> 10K
- R74: value 30K -> 750R
- R75: value 10K -> 750R
- R76: value 16K -> 30K
- R77: value 220R -> 1K8
- TP2: device EEZ_Lib1:PCB_TEST_TABSHIELD -> EEZ_Lib1:JUMPER-2PIN-2MM
- X1: device EEZ_Lib1:MINIFIT_39301039-CREEPAGE -> EEZ_connectors:MINIFIT_39301039-CREEPAGE
- X2: value B2B-ZR -> 90136-1208; device EEZ_Lib1:B2B-ZR -> con-molex:C-GRID-08-70543
- X3: value 90136-1208 -> B2B-ZR; device con-molex:C-GRID-08-70543 -> EEZ_Lib1:B2B-ZR
- X4: value B2B-ZR -> 39-28-1023; device EEZ_Lib1:B2B-ZR -> EEZ_connectors:MINIFIT_5566-02A
- ZD4: value MMSZ5V1T1G -> PDZ6.2B
- ZD5: value PDZ6.2B -> SMAJ58A-TR; device EEZ_Lib1:ZENER-DIODESOD323 -> EEZ_Lib1:PSMAXX
Connections:
- removed net ISO_FB: C46.2, IC3.COMP, OK3.COL, R50.1, TP5.P$1
- removed net N$56: Q2.D, TR2.P
- new net AGND: C34.1, C40.2, C43.1, C44.1, C45.1, C46.1, C47.2, C48.1, IC2.DISABLE, IC2.GNDI, IC3.AGND, IC3.PGND, IC4P.V-, JP4.1, OK3.EMIT, Q4.C, R19.2, R20.2, R21.2, R27.1, R27.2, R28.1, R43.2, R46.2, R47.2, R51.2, R55.2, R56.2, R57.2, R58.2, TR2.S_DOT, ZD4.A
- new net COMP: C46.2, IC3.COMP, JP8.1, R50.2
- new net N$1: D24.A, X2-4.S
- new net N$30: R41.2, R42.1
- new net N$34: C48.2, IC4A.+IN, R54.2
- new net N$39: C67.1, IC6P.V-, JP6.1
- new net N$41: B1.AC2, C2.1, C5.2, L1-2.1, SAR1.P$2
- new net N$43: B1.AC1, C2.2, C4.2, L1-1.1, SAR2.P$2
- new net N$44: JP8.2, OK3.COL
- new net N$45: C74.2, R85.1
- new net N$46: C64.1, C65.1, IC6P.V+, IC7-1.VCC+, JP5.2, R69.1, R70.1, R77.2, R79.2
- new net N$65: C44.2, IC3.REF, R38.1, R50.1
- new net NFB_IN: C73.2, IC8.REF, R78.1, R81.2, R82.2, R85.2, R86.2
- net !FAULT: now also D24.C, FAULT.C; no longer R12.2, X3-4.S
- net +12V: now also C47.1, JP1.2, R18.2, R31.2, R40.2; no longer C49.1, C6.1, Q1.E, R23.2, R34.2, R41.2, X2-1.1
- net +2.5VREF: now also R73.2, R77.1; no longer R67.2, R72.1
- net +5VREF: now also R52.2, R53.2, X3-1.1; no longer C45.2, C50.1, IC3.REF, R33.1, R51.2, X4-1.1
- net +6V_REC: now also R13.1; no longer R15.1
- net -15V: now also JP2.COM, X2-3.S; no longer JP1.COM, X3-3.S
- net 0V: now also C31.-, C32.-, C33.2, C39.1, C42.2, JP3.NO, JP4.2, Q5.S, R14.1, R15.2, R16.2, R32.2, R34.1, R34.2; no longer C28.-, C29.-, C33.1, C34.1, C39.2, C40.2, C42.1, C43.1, C44.1, C45.1, C46.1, C47.1, C48.1, C49.2, C50.2, IC2.DISABLE, IC2.GNDI, IC3.AGND, IC3.FB, IC3.PGND, IC4P.V-, JP2.NO, OK3.EMIT, Q4.S, Q5.C, R16.1, R17.2, R18.2, R20.2, R21.2, R22.2, R29.1, R29.2, R30.1, R35.2, R37.1, R37.2, R43.2, R47.2, R48.2, R52.2, R53.2, R54.2, TP1.P$1, TP4.P$1, TR2.S, X2-2.1, ZD4.A, ZD5.A
- net AC_L_IN: now also L1-2.2, X1-2.1; no longer L1-1.2, X1-1.1
- net AC_N_IN: now also L1-1.2, X1-3.1; no longer L1-2.2, X1-2.1
- net AUX_AC: now also R11.2; no longer R13.2
- net BUCK_OUT: now also C28.2, C29.2; no longer C31.2, C32.2, TP3.P$1
- net CLAMP_C: now also C39.2, D19.C, R35.1, R37.1, R42.2; no longer C43.2, C44.2, D15.C, R38.1, R39.1
- net CT_OUT: now also R20.1; no longer R22.1
- net DC_BUS: now also C31.+, C32.+, C33.1, D15.C, R30.1, TR2.P; no longer C28.+, C29.+, C33.2, R32.1, R38.2, R39.2, TR2.P_DOT
- net DC_OUT: now also X2-2.S; no longer X3-2.S
- net FB: now also IC3.FB, R41.1, R51.1, R54.1; no longer R71.1, R75.2, R76.2
- net FB2: now also R17.1; no longer R19.1
- net GND: now also C49.-, C50.-, C52.2, C53.2, C57.1, C60.1, C67.2, C72.2, IC8.A, JP2.NO, PWR.C, R65.2, R86.1, TP1.P$1, X2-6.S, X4-2.1, ZD5.A; no longer C52.-, C53.-, C57.2, C59.1, C60.2, C66.2, JP1.NO, LED1.C, R61.2, TP2.P$1, TP6.GND, X3-6.S, X5-2.1, ZD6.A
- net HD: now also R23.2; no longer R25.2
- net HI_OUT: now also D11.C, R22.2; no longer D11.A, R24.2
- net LD: now also R24.2; no longer R27.2
- net LO_OUT: now also D14.C, R29.1; no longer D14.A, R31.1
- net L_PULL: now also C38.2, D19.A, L6.P$1, TR3.P_DOT; no longer D15.A, L5.P$1, R26.2, TR3.P
- net L_PUSH: now also L5.P$1, Q5.D, R25.2, TR3.P; no longer C38.2, L6.P$1, Q4.D, TR3.P_DOT
- net N$10: now also C66.2, R76.1, R81.1; no longer C68.2, R74.1, R75.1
- net N$100: now also Q4.G, R45.1; no longer Q5.G, R46.1
- net N$11: now also PWR.A, R70.2; no longer LED1.A, R11.2
- net N$12: now also R72.1, R78.2; no longer R66.1, R71.2
- net N$126: now also Q4.A; no longer Q5.A
- net N$13: now also D20.C, Q5.G; no longer D19.C, Q4.G
- net N$130: now also R33.2; no longer LED2.C
- net N$132: now also R71.2, R73.1; no longer R65.2, R67.1
- net N$134: now also C68.1, R83.2; no longer C67.1, R77.2
- net N$135: now also R13.2; no longer R15.2
- net N$14: now also D21.C, R48.1; no longer D20.C, R45.1
- net N$141: now also R11.1, R12.1, R14.2; no longer R13.1, R14.1, R16.2
- net N$15: now also Q2.D, TR2.P_DOT; no longer B1.AC2, C2.1, C5.2, L1-1.1, SAR1.P$2
- net N$152: now also R16.1; no longer R18.1
- net N$155: now also R12.2; no longer R14.2
- net N$16: now also FAULT.A, R69.2; no longer LED2.A, R36.2
- net N$17: now also R26.1; no longer R28.1
- net N$18: now also R65.1; no longer R61.1
- net N$19: now also R47.1; no longer R48.1
- net N$2: now also R30.2, R36.1, TP2.1; no longer R32.2, R40.1
- net N$20: now also R15.1; no longer R17.1
- net N$21: now also D11.A, R22.1; no longer D11.C, R24.1
- net N$22: now also R46.1; no longer R47.1
- net N$23: now also C43.2; no longer C42.2
- net N$24: now also C6.1, JP1.1, Q1.E; no longer B1.AC1, C2.2, C4.2, L1-2.1, SAR2.P$2
- net N$25: now also R39.1, ZD4.C; no longer R42.1, ZD5.C
- net N$26: now also R52.1, R56.1; no longer R51.1, R53.1
- net N$29: now also D14.A, R29.2, R32.1; no longer D14.C, R31.2, R35.1
- net N$3: now also C28.1, C29.1; no longer C31.1, C32.1
- net N$31: now also R18.1; no longer R23.1
- net N$32: now also R33.1; no longer R36.1
- net N$35: now also D15.A, R35.2, R37.2; no longer C48.2, R50.2
- net N$36: now also R23.1; no longer R25.1
- net N$37: now also C45.2; no longer C47.2
- net N$38: now also IC4A.OUT, R45.2, R55.1; no longer R46.2, R52.1
- net N$4: now also JP3.COM; no longer JP2.COM
- net N$40: now also R24.1; no longer R27.1
- net N$42: now also R57.1, X3-2.1; no longer IC4A.-IN, IC4A.OUT
- net N$48: now also R28.2; no longer R30.2
- net N$5: now also R25.1, R26.2; no longer R26.1, R28.2
- net N$50: now also R19.1, TR2.S; no longer R20.1, TR2.S_DOT
- net N$53: now also R71.1, R74.2; no longer R65.1, R69.2
- net N$54: now also C42.1, R40.1; no longer C40.1, R41.1
- net N$57: now also C72.1, JP7.COM; no longer JP3.COM
- net N$58: now also JP7.NO; no longer JP3.NO
- net N$6: now also R64.2; no longer R60.2
- net N$63: now also R31.1; no longer R34.1
- net N$64: now also C68.2, R74.1, R75.2, R80.1; no longer C67.2, R68.2, R69.1, R73.1
- net N$66: now also C58.1, R61.2, R62.2; no longer C60.1, R57.2, R58.2
- net N$67: now also C63.1, R67.2, R68.2; no longer C64.1, R63.2, R64.2
- net N$7: now also IC4A.-IN, R53.1, R58.1; no longer IC4A.+IN, R54.1, X4-2.1
- net N$74: now also D22.C, R63.2; no longer D21.C, R59.2
- net N$75: now also D23.C, R66.2; no longer D22.C, R62.2
- net N$76: now also C66.1, C73.1, C74.1, IC8.C, R84.2; no longer C68.1
- net N$8: now also C57.2, R60.1; no longer C59.2, R56.1
- net N$9: now also R76.2; no longer R74.2
- net NFB_OFFSET: now also R75.1, R82.1, R83.1; no longer R68.1, R76.1, R77.1
- net OK_A: now also R79.1, R84.1; no longer R70.1
- net PE: now also C59.2, C60.2, JP3.NC, X1-1.1, X2-8.S; no longer JP2.NC, X1-3.1, X3-8.S
- net POUT+: now also C49.+, C50.+, C52.1, R59.1, R72.2; no longer C52.+, C53.+, C54.1, R55.1, R66.2
- net PREG_OUT+: now also C53.1, C54.1, C59.1, JP2.NC, R59.2, R60.2, X4-1.1, ZD5.C; no longer C57.1, C58.1, JP1.NC, R55.2, R56.2, TP6.TIP, X5-1.1, ZD6.C
- net PULL: now also D21.A, R48.2; no longer D20.A, R45.2
- net PUSH: now also D20.A; no longer D19.A
- net REF: now also R38.2; no longer R33.2, ZD4.C
- net S1_DOT_OUT: now also R61.1, R62.1; no longer R57.1, R58.1
- net S2_OUT: now also R67.1, R68.1; no longer R63.1, R64.1
- net SR_OUT1: now also D22.A, R63.1; no longer D21.A, R59.1
- net SR_OUT2: now also D23.A, R66.1; no longer D22.A, R62.1
- net ULVO: now also C40.1, R36.2, R39.2, TP2.2; no longer C39.1, R40.2, R42.2
- net U_MON: now also JP7.NC, X2-1.S; no longer JP3.NC, X3-1.S
- net U_MON1: now also R80.2; no longer R73.2
- net V+: now also JP5.1, R17.2, R64.1, X2-5.S; no longer C63.1, C66.1, IC6P.V+, IC7-1.VCC+, R11.1, R12.1, R19.2, R60.1, R70.2, R72.2, X3-5.S
- net V-: now also JP6.2, X2-7.S; no longer C65.1, IC6P.V-, X3-7.S
Other:
- note added: "+23 V"
- note added: "+6.5 V"
- note added: "-8 V"
- note added: "0R"
- note added: "100K"
- note added: "2:1:1 (30/15/15 turns)"
- note added: "2K2"
- note added: "4K7"
- note added: "Current-fed dual inductor converter (CF-DIC) Overvotlage and Overtemperature protection"
- note added: "Max. +2.5V"
- note added: "OVP and OTP"
- note added: "Pri 30 turns, Sec 2 x 15"
- note added: "Pri: Ø 0.4 mm x 3 + CB-HFT2.4"
- note added: "Sec: Ø 0.4 mm x 6"
- note added: "Use TP2 jumper for Vin below 120 Vdc"
- note added: "X1 3-pin input connector"
- note added: "X2 8-pin output connector"
- note removed: ""Fault" (red)"
- note removed: ""Power" (yellow)"
- note removed: "(e.g. 28/16/16 turns)"
- note removed: "(optional)"
- note removed: "1.75:1:1 to 2:1:1"
- note removed: "16K"
- note removed: "3-31.5V"
- note removed: "3-41.5V"
- note removed: "3-51.5V"
- note removed: "328K"
- note removed: "Current-fed dual inductor converter (CF-DIC)"
- note removed: "Default range: 50 V"
- note removed: "Murata 680 uH"
- note removed: "R65+R71"
- note removed: "R76"
- note removed: "Range"
- note removed: "Route traces between PP MOSFETs and transformer primary as short as possible and of equal length"
- note removed: "TBA"
- note removed: "Thermal protection"
- note removed: "X2 3-pin input connector"
- note removed: "X3 8-pin output connector"
- note removed: "fsw = 66 kHz @ Rt = 82K"
- moved on the sheet: B1, C1, C19, C2, C20, C22, C26, C27, C30, C33, C34, C35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

Commit message: X2 rotated for easier cable insertion
Parts:
- X2: device con-molex:C-GRID-08-70543 -> EEZ_connectors:C-GRID-08-70543
Connections:
- net -15V: now also X2-6.S; no longer X2-3.S
- net DC_OUT: now also X2-7.S; no longer X2-2.S
- net GND: now also X2-3.S; no longer X2-6.S
- net N$1: now also X2-5.S; no longer X2-4.S
- net PE: now also X2-1.S; no longer X2-8.S
- net U_MON: now also X2-8.S; no longer X2-1.S
- net V+: now also X2-4.S; no longer X2-5.S
- net V-: now also X2-2.S; no longer X2-7.S
Other:
- note added: "!FAULT! 5"
- note added: "Bias+ 7"
- note added: "Bias- 6"
- note added: "GND 3"
- note added: "PE 1"
- note added: "U_MON 8"
- note added: "V+ 4"
- note added: "V- 2"
- note removed: "!FAULT! 4"
- note removed: "Bias+ 2"
- note removed: "Bias- 3"
- note removed: "GND 6"
- note removed: "PE 8"
- note removed: "U_MON 1"
- note removed: "V+ 5"
- note removed: "V- 7"
- moved on the sheet: X2-2, X2-3, X2-6, X2-7
