File: Eagle files/EEZ CF-DIC r5B5.sch (EAGLE design)
At the start: 245 parts, among them IC1 VIPer35L, IC2 SI8233BB-D-IS1, IC3 LM5041B, IC4 LM258D, IC5 IR11688STRPBF, IC6 TL072, IC7 TL103W, IC8 TL431, P1 T910W-50K, Q1 MMBT5551, Q2 C3M0280090D, Q3 C3M0280090D, Q4 NYC0102BLT1G, Q5 C3M0280090D, Q6 C3M0280090D, Q7 IRFS4321PBF, Q8 IRFS4321PBF, X1 39-30-1039, X2 90136-1208, X3 B2B-ZR, X4 39-28-1023

Commit message: r5B5 version
Parts:
- removed FAULT: LTST-C170KRKT, EEZ_Lib1:LED0805
- removed IC8: TL431, EEZ_Lib1:TL431
- removed PWR: LTST-C170YKT, EEZ_Lib1:LED0805
- added C75: 2n2, rcl:C-EUC0805
- added C76: 4u7, EEZ_Lib1:ECAP1206
- added C77: 1u, rcl:C-EUC0805
- added C78: N.C., rcl:C-EUC0805
- added D25, D26: 1N5819HW-7-F, diode:DIODE-SOD323-W
- added D27: BAS316, EEZ_Lib1:DIODESOD323R
- added LED1: L-934EB/1Y1ID-RV, EEZ_Lib1:LED_L-934EB/1Y1ID-RV
- added R87: 10K, rcl:R-EU_R0805
- added R88: 7K5, rcl:R-EU_R0805
- added R89: 220R, rcl:R-EU_R0805
- added TP3, TP4, TP5: (no value), EEZ_connectors:TEST-PIN1.2
- added TP6: (no value), EEZ_Lib1:TEST_POINT-2
- C15, C22: device rcl:C-EUC1210 -> rcl:C-EUC1206
- C20: value 470u -> 1500u
- C31, C32: value UCY2G121MHD -> UPH2G151MHD6
- C40: value 10n -> 100n; device rcl:C-EUC0805 -> rcl:C-EUC0603
- C43: value 10n -> 1u
- C44: value 100n -> 10n
- C45: value 1n -> 100n; device rcl:C-EUC0805 -> rcl:C-EUC0603
- C46: value 100p -> 470p
- C47: value 100n -> 470p; device rcl:C-EUC0603 -> rcl:C-EUC0805
- C48: value 1u -> 10n; device rcl:C-EUC0805 -> rcl:C-EUC0603
- C49, C51: value UPW1J152MHD -> 100n; device EEZ_Lib1:ECAP7.5G_18MM -> rcl:C-EUC0603
- C4A: device EEZ_Lib1:C-EUCY -> EEZ_Lib1:C-EUCY-ROTATED
- C50: value UPW1J152MHD -> 1u; device EEZ_Lib1:ECAP7.5G_18MM -> rcl:C-EUC0805
- C52: value 1u/100V -> N.C.; device rcl:C-EUC1206 -> rcl:C-EUC0603
- C53: value HHXC630ARA330MHA0G -> 1u; device Panasonic-EEEFK_EEEFP:EEE-FK1J470P-CASE-F -> rcl:C-EUC0805; MPN EEE-FK1J470P -> (none); OC_FARNELL 9696032 -> (none); OC_NEWARK 96K9403 -> (none); PACKAGE CASE-F -> (none); SUPPLIER PANASONIC -> (none); TOLERANCE ±20 % -> (none); VALUE 47UF -> (none); VOLTAGERATING 63 V -> (none)
- C54: value HHXC630ARA330MHA0G -> UPW1J152MHD; device Panasonic-EEEFK_EEEFP:EEE-FK1J470P-CASE-F -> EEZ_Lib1:ECAP7.5G_18MM
- C55: value 1u/100V -> UPW1J152MHD; device rcl:C-EUC1206 -> EEZ_Lib1:ECAP7.5G_18MM
- C56: value 100n/100V -> UPW1J152MHD; device rcl:C-EUC1206 -> EEZ_Lib1:ECAP7.5G_18MM
- C57, C60: value N.C. -> 1u/100V
- C58: value 4n7/200V -> HHXC630ARA330MHA0G; device rcl:C-EUC1206 -> EEZ_Lib1:ECAPSMD8.3MM/HA0
- C59: device rcl:C-EUC1206 -> EEZ_Lib1:ECAPSMD8.3MM/HA0
- C61: value 100n -> 100n/100V; device rcl:C-EUC0603 -> rcl:C-EUC1206
- C62: value 4u7 -> N.C.
- C65: value 100n -> 4u7; device rcl:C-EUC0603 -> rcl:C-EUC1206
- C66, C68: value 100p -> 4n7/200V; device rcl:C-EUC0805 -> rcl:C-EUC1206
- C67: value 100n -> 4n7/200V; device rcl:C-EUC0603 -> rcl:C-EUC1206
- C69: value 33n -> 100n; device rcl:C-EUC0805 -> rcl:C-EUC0603
- C70: value 4u7 -> 10n; device EEZ_Lib1:ECAP1206 -> rcl:C-EUC0603
- C71: value 1u -> 100n; device rcl:C-EUC0805 -> rcl:C-EUC0603
- C72: value N.C. -> 100p
- C73: value N.C. -> 100n; device rcl:C-EUC0805 -> rcl:C-EUC0603
- C74: value 1n -> 100p
- C8: value 470n -> 1u
- D10: value C3D02065E -> 1N5819HW-7-F; device EEZ_Lib1:SCHOTTKY-SIC -> diode:DIODE-SOD323-W
- D11: value N.C. -> C3D06065A; device diode:DIODE-SOD323-W -> EEZ_Lib1:SCHOTTKY-TO220
- D12: value C3D06065A -> 1N5819HW-7-F; device EEZ_Lib1:SCHOTTKY-TO220 -> diode:DIODE-SOD323-W
- D14: value N.C. -> US1K-DIO; device diode:DIODE-SOD323-W -> EEZ_Lib1:DIODEDO214AA
- D15: value US1M-DIO -> C3D02065E; device EEZ_Lib1:DIODEDO214AA -> EEZ_Lib1:SCHOTTKY-SIC
- D16: value C3D02065E -> BAS316; device EEZ_Lib1:SCHOTTKY-SIC -> EEZ_Lib1:DIODESOD323R
- D18, D9: value BAS316 -> C3D02065E; device EEZ_Lib1:DIODESOD323R -> EEZ_Lib1:SCHOTTKY-SIC
- D19: value C3D02065E -> N.C.; device EEZ_Lib1:SCHOTTKY-SIC -> diode:DIODE-SOD323-W
- D20, D22, D23: value 1N5819HW-7-F -> BAS316; device diode:DIODE-SOD323-W -> EEZ_Lib1:DIODESOD323R
- D21: value 1N5819HW-7-F -> N.C.
- IC6: value TL072 -> LM258D
- Q7, Q8: value IRFS4321PBF -> FDD86250-F085
- R20: value 6R2 -> 33R
- R21: value N.C. -> 10R
- R22: value 10R -> 100R
- R24: value 100R -> 22R/2-3W; device rcl:R-EU_R0805 -> rcl:R-EU_R2512
- R26: value 22R/2-3W -> 1R; device rcl:R-EU_R2512 -> rcl:R-EU_R0805
- R27: value 1R -> 30K
- R28: value 30K -> 33R
- R29: value 10R -> 220K; device rcl:R-EU_R0805 -> rcl:R-EU_R1206
- R30: value 220K -> 10R; device rcl:R-EU_R1206 -> rcl:R-EU_R0805
- R33: value 1K -> 1R
- R34: value 1R -> 22R/2-3W; device rcl:R-EU_R0805 -> rcl:R-EU_R2512
- R35, R61, R62: value 22R/2-3W -> 1K; device rcl:R-EU_R2512 -> rcl:R-EU_R0805
- R41: value 30K -> 10K
- R42: value 100K -> 30K
- R43: value 10K -> 100K
- R44: value 22R -> 33R
- R45: value 4K7 -> 30K
- R46: value 33K -> 82K
- R47: value 51K -> 33R
- R48: value 22R -> 1K
- R49: value 1K -> N.C.
- R50: value N.C. -> 6R2
- R51: value 750R -> 4K7
- R52: value 4K7 -> 750R
- R53: value 5K6 -> 1K
- R54: value 30K -> 8K2
- R55: value 1K -> 4K7
- R56: value 30K -> 5K6
- R57: value 10K -> 47K
- R59: value 120R -> 30K
- R60: value N.C. -> 10K; device rcl:R-EU_R1210 -> rcl:R-EU_R0805
- R63: value 3R3 -> 120R
- R64: value 10R -> N.C.; device rcl:R-EU_R0805 -> rcl:R-EU_R1210
- R65: value 47K -> 22R/2-3W; device rcl:R-EU_R0805 -> rcl:R-EU_R2512
- R66: value 3R3 -> 22R/2-3W; device rcl:R-EU_R0805 -> rcl:R-EU_R2512
- R67: value 22R/2-3W -> 47K; device rcl:R-EU_R2512 -> rcl:R-EU_R0805
- R68: value 22R/2-3W -> 3R3; device rcl:R-EU_R2512 -> rcl:R-EU_R0805
- R69: value 470R -> 10R
- R70: value 470R -> 47K
- R71: value 10K -> 3R3
- R72: value 316K -> 22R/2-3W; device rcl:R-EU_R0805 -> rcl:R-EU_R2512
- R73: value 10K -> 22R/2-3W; device rcl:R-EU_R0805 -> rcl:R-EU_R2512
- R74: value 750R -> 10K
- R75, R80: value 750R -> 470R
- R76: value 30K -> 470R
- R77: value 1K8 -> 100K
- R78: value 12K -> 10K
- R79: value 470R -> 750R
- R81: value 10K -> 51K
- R82: value 16K -> 750R
- R83: value 220R -> 30K
- R84: value 750R -> 1K8
- R85: value 6K8 -> 3K3
- R86: value 7K5 -> 750R
- X1: value 39-30-1039 -> 39-30-3035; device EEZ_connectors:MINIFIT_39301039-CREEPAGE -> EEZ_connectors:MINIFIT_6659-3-CRE
- X2: value 90136-1208 -> 22-05-7085; device EEZ_connectors:C-GRID-08-70543 -> EEZ_connectors:SPOX_22-05-7085
- X4: value 39-28-1023 -> 39-30-1020; device EEZ_connectors:MINIFIT_5566-02A -> EEZ_connectors:MINIFIT_39301020
- ZD4: value PDZ6.2B -> MMSZ5V1T1G
Connections:
- removed net CT_OUT: D9.C, R20.1, R21.1, R49.1
- removed net N$65: C44.2, IC3.REF, R38.1, R50.1
- removed net NFB_IN: C73.2, IC8.REF, R78.1, R81.2, R82.2, R85.2, R86.2
- new net CT_OUT+: D20.A, R19.1, TR2.S
- new net CT_OUT-: R19.2, R50.2, R53.1, TR2.S_DOT
- new net N$28: C70.2, R80.2
- new net N$47: D24.A, IC4B.OUT
- new net N$51: D22.C, D24.C, R51.2, R58.1
- new net N$52: D13.C, R31.2
- new net N$56: D20.C, R48.1, R50.1
- new net N$59: C50.2, D23.A, R62.1
- net !FAULT: now also D27.C, LED1-BTM.C; no longer D24.C, FAULT.C
- net +12V: now also C49.1, C50.1, R30.2; no longer C47.1, R31.2
- net +2.5VREF: now also C77.1, R78.2, R84.1; no longer C71.1, R73.2, R77.1
- net +5VREF: now also C45.2, IC3.REF, R38.1, R49.1, R55.2, R56.2, X3-2.1; no longer R52.2, R53.2, X3-1.1
- net -15V: now also X2-7.1; no longer X2-6.S
- net 0V: now also D11.A, R33.1, R33.2, TP3.P$1, TP4.P$1, TP5.P$1; no longer D12.A, R34.1, R34.2
- net AC_L_IN: now also C1.2, C5A.2, L1-1.2, R2.2, SAR2.P$1, X1-1.1; no longer C1.1, C4A.2, L1-2.2, R1.1, SAR1.P$1, X1-2.1
- net AC_N_IN: now also C1.1, C4A.2, L1-2.2, R1.1, SAR1.P$1, X1-2.1; no longer C1.2, C5A.2, L1-1.2, R2.2, SAR2.P$1, X1-3.1
- net AGND: now also C44.2, C47.1, C48.2, C49.2, C51.2, C52.1, C53.1, R26.1, R26.2, R41.2, R45.2, R52.2, R53.2, R54.1, R59.2, R60.2, R61.2, R62.2; no longer C44.1, C47.2, C48.1, R19.2, R20.2, R21.2, R27.2, R28.1, R43.2, R47.2, R51.2, R55.2, R56.2, R57.2, TR2.S_DOT
- net BUCK_OUT: now also D11.C; no longer D12.C
- net CLAMP_C: now also D15.C, D18.C, R34.1, R43.2; no longer D16.C, D19.C, R35.1, R42.2
- net COMP: now also C47.2, R49.2, R54.2; no longer C46.2, R50.2
- net DC_BUS: now also D14.C, R29.1; no longer D15.C, R30.1
- net DC_OUT: now also X2-8.1; no longer X2-7.S
- net FB: now also C48.1, R42.1, R52.1, R57.1; no longer R41.1, R51.1, R54.1
- net GND: now also C54.-, C55.-, C56.-, C57.2, C58.-, C59.-, C60.2, C62.1, C67.1, C68.2, C69.2, C73.2, C76.-, C77.2, C78.2, LED1-TOP.C, R67.1, R70.2, TP6.GND, X2-2.1, X2-6.1; no longer C49.-, C50.-, C51.-, C52.2, C53.2, C54.2, C55.2, C56.2, C57.1, C58.2, C60.1, C62.2, C67.2, C70.-, C72.2, IC8.A, PWR.C, R65.2, R86.1, X2-3.S
- net HD: now also R22.2; no longer R23.2
- net HI_OUT: now also R20.2, R21.2; no longer D11.C, R22.2
- net LD: now also R23.2; no longer R24.2
- net LO_OUT: now also R28.1, R31.1; no longer D14.C, R29.1
- net L_PULL: now also D18.A; no longer D19.A
- net L_PUSH: now also D15.A, R24.2; no longer D16.A, R25.2
- net N$1: now also D27.A, X2-4.1; no longer D24.A, X2-5.S
- net N$10: now also C72.2, R83.1, R87.1; no longer C66.2, R76.1, R81.1
- net N$100: now also C44.1, R51.1; no longer R45.1
- net N$11: now also LED1-TOP.A, R76.2; no longer PWR.A, R70.2
- net N$12: now also R77.1, R81.2; no longer R72.1, R78.2
- net N$126: now also D16.C; no longer D18.C
- net N$13: now also D19.C; no longer D20.C
- net N$130: now also D16.A, R35.2; no longer D17.A, R33.2
- net N$132: now also R74.2, R78.1; no longer R71.2, R73.1
- net N$134: now also C74.1, R89.2; no longer C68.1, R83.2
- net N$14: now also R47.1; no longer R48.1
- net N$16: now also LED1-BTM.A, R75.2; no longer FAULT.A, R69.2
- net N$17: now also R25.1; no longer R26.1
- net N$18: now also R70.1; no longer R65.1
- net N$19: now also R46.1; no longer R47.1
- net N$2: now also R29.2; no longer R30.2
- net N$21: now also D10.A, R20.1; no longer D11.A, R22.1
- net N$22: now also R45.1; no longer R46.1
- net N$25: now also C40.1
- net N$26: now also R55.1, R59.1; no longer R52.1, R56.1
- net N$29: now also D13.A, R28.2; no longer D14.A, R29.2
- net N$3: now also D9.C; no longer D10.C
- net N$30: now also R42.2, R43.1; no longer R41.2, R42.1
- net N$31: now also D9.A; no longer D10.A
- net N$32: now also R35.1; no longer R33.1
- net N$34: now also C53.2, R57.2; no longer C48.2, R54.2
- net N$35: now also D14.A, R34.2; no longer D15.A, R35.2
- net N$36: now also R22.1; no longer R23.1
- net N$37: now also C46.2, R48.2; no longer C45.2, R49.2
- net N$38: now also D22.A; no longer IC4B.OUT, R45.2, R55.1
- net N$39: now also C73.1; no longer C67.1
- net N$40: now also R23.1; no longer R24.1
- net N$41: now also B1.AC1; no longer B1.AC2
- net N$42: now also C52.2, R60.1, X3-1.1; no longer R57.1, X3-2.1
- net N$43: now also B1.AC2; no longer B1.AC1
- net N$45: now also D10.C, R21.1; no longer C74.2, R85.1
- net N$46: now also C69.1, C71.1, R84.2, R85.2; no longer C64.1, C65.1, R70.1, R77.2, R79.2
- net N$48: now also R27.2; no longer R28.2
- net N$5: now also R24.1, R25.2; no longer R25.1, R26.2
- net N$50: now also R80.1, R81.1, R87.2, R88.2; no longer D9.A, R19.1, TR2.S
- net N$53: now also R74.1, R79.2; no longer R71.1, R74.2
- net N$55: now also D12.C; no longer D13.C
- net N$57: now also C78.1; no longer C72.1
- net N$6: now also C64.1, C65.1, R69.2; no longer C61.1, C62.1, R64.2
- net N$63: now also D12.A, R30.1; no longer D13.A, R31.1
- net N$64: now also C74.2, R79.1, R82.2, R86.1; no longer C68.2, R74.1, R75.2, R80.1
- net N$66: now also C63.1, R65.2, R66.2; no longer C58.1, R61.2, R62.2
- net N$67: now also C68.1, R72.2, R73.2; no longer C63.1, R67.2, R68.2
- net N$7: now also C51.1, D23.C, R56.1, R61.1; no longer R53.1, R58.1
- net N$74: now also D25.C, R68.2; no longer D22.C, R63.2
- net N$75: now also D26.C, R71.2; no longer D23.C, R66.2
- net N$76: now also C72.1, C75.1; no longer C66.1, C69.1, C73.1, C74.1, IC8.C, R84.2
- net N$8: now also C62.2, R64.1; no longer C57.2, R60.1
- net N$9: now also C75.2, R83.2; no longer C69.2, R76.2
- net NFB_OFFSET: now also C76.+, R88.1, R89.1; no longer C70.+, R75.1, R83.1
- net OK_A: now also R85.1; no longer R79.1, R84.1
- net PE: now also C66.2, C67.2, X1-3.1; no longer C59.2, C60.2, X1-1.1, X2-1.S
- net POUT+: now also C54.+, C55.+, C56.+, C57.1, R63.1; no longer C49.+, C50.+, C51.+, C52.1, R59.1, R72.2
- net PREG_OUT+: now also C58.+, C59.+, C60.1, C61.1, C66.1, C70.1, R63.2, R64.2, R67.2, R77.2, TP6.TIP; no longer C53.1, C54.1, C55.1, C56.1, C59.1, R59.2, R60.2
- net PULL: now also R47.2; no longer R48.2
- net PUSH: now also D19.A; no longer D20.A
- net S1_DOT_OUT: now also R65.1, R66.1; no longer R61.1, R62.1
- net S2_OUT: now also R72.1, R73.1; no longer R67.1, R68.1
- net SR_OUT1: now also D25.A, R68.1; no longer D22.A, R63.1
- net SR_OUT2: now also D26.A, R71.1; no longer D23.A, R66.1
- net ULVO: now also D17.A, R41.1; no longer C40.1, D18.A, R43.1
- net U_MON: now also X2-5.1; no longer X2-8.S
- net U_MON1: now also R86.2; no longer R80.2
- net V+: now also R75.1, R76.1, X2-3.1; no longer R64.1, X2-4.S
- net V-: now also X2-1.1; no longer X2-2.S
Other:
- note added: "!FAULT! 4"
- note added: "1.875:1:1 (30/16/16 turns)"
- note added: "Bias+ 8"
- note added: "Bias- 7"
- note added: "Current-fed dual inductor converter (CF-DIC) OTP, OVP/short-circuit protection"
- note added: "NTCALUG03A103HC (10K NTC)"
- note added: "OTP trip set to ~73oC (+4.32 V) for selected NTC (10K/3984K). Decrease R53 to 2K7 for ~90oC."
- note added: "Place OK3 as close as possible to IC3"
- note added: "Repository: https://github.com/eez-open/CF-DIC"
- note added: "Route traces between sync. MOSFETs and transformer outputs as short as possible"
- note added: "U_MON+ 5"
- note added: "U_MON- 6"
- note added: "Use TP2 jumper for testing purposes only when DC_BUS is below ~85 Vdc"
- note added: "V+ 3"
- note added: "V- 1"
- note removed: "!FAULT! 5"
- note removed: "0R"
- note removed: "100K"
- note removed: "2:1:1 (30/15/15 turns)"
- note removed: "2K2"
- note removed: "4K7"
- note removed: "Bias+ 7"
- note removed: "Bias- 6"
- note removed: "Current-fed dual inductor converter (CF-DIC) Overvotlage and Overtemperature protection"
- note removed: "GND 3"
- note removed: "PE 1"
- note removed: "Pri 30 turns, Sec 2 x 15"
- note removed: "Repository: https://github.com/eez-open"
- note removed: "Route traces between sync. MOSFETs and transformer outputs as shoort as possible"
- note removed: "U_MON 8"
- note removed: "Use TP2 jumper for Vin below 120 Vdc"
- note removed: "V+ 4"
- note removed: "V- 2"
- moved on the sheet: B1, C26, C27, C28, C29, C30, C31, C32, C33, C34, C35, C36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

Commit message: C4, C5, C17 value changed
Parts:
- C17, C4, C5: value CY1Y-470P -> CY1Y-4N7
Changed lines of the file:
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@@
 <setting verticaltext="up"/>
 </settings>
-<grid distance="0.1" unitdist="inch" unit="inch" style="lines" multiple="1" display="no" altdistance="0.01" altunitdist="inch" altunit="inch"/>
+<grid distance="0.025" unitdist="inch" unit="inch" style="lines" multiple="4" display="no" altdistance="0.01" altunitdist="inch" altunit="inch"/>
 <layers>
 <layer number="1" name="Top" color="4" fill="1" visible="no" active="no"/>
@@
 <part name="X1" library="EEZ_connectors" deviceset="MINIFIT_6659-3" device="-CRE" value="39-30-3035"/>
 <part name="PE1" library="supply1" deviceset="PE" device=""/>
-<part name="C5" library="EEZ_Lib1" deviceset="C-EU" device="CY" value="CY1Y-470P"/>
-<part name="C4" library="EEZ_Lib1" deviceset="C-EU" device="CY" value="CY1Y-470P"/>
+<part name="C5" library="EEZ_Lib1" deviceset="C-EU" device="CY" value="CY1Y-4N7"/>
+<part name="C4" library="EEZ_Lib1" deviceset="C-EU" device="CY" value="CY1Y-4N7"/>
 <part name="R1" library="rcl" deviceset="R-EU_" device="R1206" value="220K"/>
 <part name="SAR2" library="EEZ_Lib1" deviceset="SAR" device="PCB-2.4MM" value="PCB 2.4mm"/>
@@
 <part name="R4" library="rcl" deviceset="R-EU_" device="R0805" value="1K8"/>
 <part name="C6" library="rcl" deviceset="C-EU" device="C0603" value="N.C."/>
-<part name="C17" library="EEZ_Lib1" deviceset="C-EU" device="CY" value="CY1Y-470P"/>
+<part name="C17" library="EEZ_Lib1" deviceset="C-EU" device="CY" value="CY1Y-4N7"/>
 <part name="C8" library="rcl" deviceset="C-EU" device="C0805" value="1u"/>
 <part name="OK1" library="EEZ_Lib1" deviceset="TLP291" device="" value="TLP291-GB.SE-T"/>
@@
 </instance>
 <instance part="C5" gate="G$1" x="73.66" y="139.7" smashed="yes" rot="R180">
-<attribute name="NAME" x="75.819" y="140.716" size="1.778" layer="95"/>
-<attribute name="VALUE" x="75.819" y="138.811" size="1.27" layer="96"/>
+<attribute name="NAME" x="75.819" y="141.351" size="1.778" layer="95"/>
+<attribute name="VALUE" x="75.819" y="138.811" size="1.778" layer="96"/>
 </instance>
 <instance part="C4" gate="G$1" x="66.04" y="139.7" smashed="yes" rot="R180">
-<attribute name="NAME" x="63.881" y="140.716" size="1.778" layer="95" rot="MR0"/>
-<attribute name="VALUE" x="63.881" y="138.811" size="1.27" layer="96" rot="MR0"/>
+<attribute name="NAME" x="63.881" y="141.351" size="1.778" layer="95" rot="MR0"/>
+<attribute name="VALUE" x="63.881" y="138.811" size="1.778" layer="96" rot="MR0"/>
 </instance>
 <instance part="R1" gate="G$1" x="30.48" y="162.56" smashed="yes" rot="R270">

Commit message: Mechanical drawings, optional EMI parts
Parts:
- added C79: N.C., rcl:C-EUC0805
- added JP9: JP2-NOCUT, EEZ_Lib1:JP2-NOCUT
- added L8: IHLP2020CZER3R3M11, EEZ_inductors_and_transformers:IHLP-2020BZ-11
- C69: value 100n -> 4n7/200V; device rcl:C-EUC0603 -> rcl:C-EUC1206
- C70: value 10n -> 100n
- C71: value 100n -> 10n
- C72, C74: value 100p -> 100n; device rcl:C-EUC0805 -> rcl:C-EUC0603
- C73: value 100n -> 100p; device rcl:C-EUC0603 -> rcl:C-EUC0805
- C75: value 2n2 -> 100p
- C76: value 4u7 -> 2n2; device EEZ_Lib1:ECAP1206 -> rcl:C-EUC0805
- C77: value 1u -> 4u7; device rcl:C-EUC0805 -> EEZ_Lib1:ECAP1206
- C78: value N.C. -> 1u
- JP2, JP7: value JP3-CUT -> JP2-NOCUT; device EEZ_Lib1:JP3-CUT -> EEZ_Lib1:JP2-NOCUT
- JP4, JP8: value JP2-NOCUT -> JP3-CUT; device EEZ_Lib1:JP2-NOCUT -> EEZ_Lib1:JP3-CUT
- L3: value DLG-0403-180 -> RLB0812-471KL; device EEZ_inductors_and_transformers:DE0403 -> EEZ_Lib1:FERYSTER_DSZ6
- L5: value 60B684C -> DLG-0403-180; device EEZ_inductors_and_transformers:MURATA_6000B -> EEZ_inductors_and_transformers:DE0403
- L7: value IHLP2020CZER3R3M11 -> 60B684C; device EEZ_inductors_and_transformers:IHLP-2020BZ-11 -> EEZ_inductors_and_transformers:MURATA_6000B
Connections:
- new net VIPER+: C12.1, C13.+, JP2.2, L3.2, R6.1, R7.1, TR1.P, TR1.SHIELD
- net +2.5VREF: now also C78.1; no longer C77.1
- net +6V_REC: now also L5.1; no longer L4.1
- net -15V: now also JP3.COM; no longer JP2.COM
- net -7V_REC: now also L4.1; no longer L3.1
- net 0V: now also JP4.NO, JP5.2; no longer JP3.NO, JP4.2
- net AGND: now also JP5.1; no longer JP4.1
- net BUCK_OUT: now also L7.P$2; no longer L5.P$2
- net COMP: now also JP9.1; no longer JP8.1
- net DC_BUS: now also JP2.1, L3.1; no longer C12.1, C13.+, R6.1, R7.1, TR1.P, TR1.SHIELD
- net GND: now also C68.1, C70.2, C72.2, C74.2, C77.-, C79.2, JP3.NO; no longer C67.1, C68.2, C71.2, C73.2, C76.-, C77.2, JP2.NO
- net L_PULL: now also L7.P$1; no longer L6.P$1
- net L_PUSH: now also L6.P$1; no longer L5.P$1
- net N$10: now also C73.2; no longer C72.2
- net N$134: now also C75.1; no longer C74.1
- net N$28: now also C71.2; no longer C70.2
- net N$39: now also C74.1, JP7.1; no longer C73.1, JP6.1
- net N$4: now also JP4.COM; no longer JP3.COM
- net N$44: now also JP9.2; no longer JP8.2
- net N$46: now also C70.1, C72.1, JP6.2; no longer C69.1, C71.1, JP5.2
- net N$57: now also C79.1, JP8.COM; no longer C78.1, JP7.COM
- net N$58: now also JP8.NO; no longer JP7.NO
- net N$64: now also C75.2; no longer C74.2
- net N$67: now also C69.1; no longer C68.1
- net N$76: now also C73.1, C76.1; no longer C72.1, C75.1
- net N$9: now also C76.2; no longer C75.2
- net NFB_OFFSET: now also C77.+; no longer C76.+
- net PE: now also C68.2, JP4.NC; no longer JP3.NC
- net POUT+: now also C66.1, L8.1; no longer L7.1
- net PREG_OUT+: now also C67.1, C71.1, JP3.NC, L8.2; no longer C66.1, C70.1, JP2.NC, L7.2
- net U_MON: now also JP8.NC; no longer JP7.NC
- net V+: now also JP6.1, L5.2; no longer JP5.1, L4.2
- net V-: now also JP7.2, L4.2; no longer JP6.2, L3.2
Other:
- moved on the sheet: C66, C67, C68, C69, C70, C71, C72, C73, C74, C75, C78, JP3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

Commit message: C46 increased to 2n2 (Eagle files)
Parts:
- C46: value 470p -> 2n2
Other:
- note added: "OTP trip set to ~73oC (+4.32 V) for selected NTC (10K/3984K). Decrease R55 to 2K7 for ~90oC."
- note added: "Rct"
- note removed: "OTP trip set to ~73oC (+4.32 V) for selected NTC (10K/3984K). Decrease R53 to 2K7 for ~90oC."
Changed lines of the file:
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@@
 <part name="D11" library="EEZ_Lib1" deviceset="SCHOTTKY" device="-TO220" value="C3D06065A"/>
 <part name="R48" library="rcl" deviceset="R-EU_" device="R0805" value="1K"/>
-<part name="C46" library="rcl" deviceset="C-EU" device="C0805" value="470p"/>
+<part name="C46" library="rcl" deviceset="C-EU" device="C0805" value="2n2"/>
 <part name="R32" library="rcl" deviceset="R-EU_" device="R0805" value="47K"/>
 <part name="R24" library="rcl" deviceset="R-EU_" device="R2512" value="22R/2-3W"/>
@@
 (10K NTC)</text>
 <text x="63.5" y="7.62" size="1.27" layer="103" align="top-left">OTP trip set to ~73oC (+4.32 V) for selected NTC (10K/3984K).
-Decrease R53 to 2K7 for ~90oC.</text>
+Decrease R55 to 2K7 for ~90oC.</text>
 <rectangle x1="70.485" y1="12.7" x2="76.2" y2="20.32" layer="97"/>
 <rectangle x1="199.39" y1="84.455" x2="207.645" y2="88.9" layer="97"/>
 <rectangle x1="199.39" y1="63.5" x2="207.645" y2="67.945" layer="97"/>
 <rectangle x1="61.595" y1="61.595" x2="69.85" y2="66.04" layer="97"/>
+<text x="143.51" y="57.15" size="1.27" layer="100">Rct</text>
 </plain>
 <instances>
