File: Eagle files/EEZ CF-DIC r5B6.brd (EAGLE design)
At the start: 155 x 90 mm, 278 parts, among them IC1 VIPer35L, IC2 SI8233BB-D-IS1, IC3 LM5041B, IC4 LM258D, IC5 IR11688STRPBF, IC6 LM258D, IC7 TL103W, P1 T910W-50K, Q1 MMBT5551, Q10 BC856C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

Commit message: 7V secondary wiring fix
Connections:
- net 6VAC: no longer TR1.9
- net 7VAC: now also TR1.9; no longer TR1.11
- net GND: now also TR1.11
Routing:
- net 6VAC: track 28.7 -> 18.9 mm
- net 7VAC: track 33.1 -> 37.3 mm
Changed lines of the file:
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@@
 <layer number="17" name="Pads" color="14" fill="1" visible="yes" active="yes"/>
 <layer number="18" name="Vias" color="6" fill="1" visible="yes" active="yes"/>
-<layer number="19" name="Unrouted" color="6" fill="1" visible="no" active="yes"/>
+<layer number="19" name="Unrouted" color="6" fill="1" visible="yes" active="yes"/>
 <layer number="20" name="Dimension" color="4" fill="1" visible="yes" active="yes"/>
 <layer number="21" name="tPlace" color="7" fill="1" visible="yes" active="yes"/>
@@
 <vertex x="113.7285" y="36.3855"/>
 </polygon>
-<wire x1="101.0285" y1="24.4475" x2="127.889" y2="24.4475" width="1.27" layer="16"/>
-<wire x1="99.247" y1="21.9405" x2="99.247" y2="16.637" width="1.27" layer="16"/>
+<wire x1="103.251" y1="24.4475" x2="127.889" y2="24.4475" width="1.27" layer="16"/>
 <wire x1="99.247" y1="16.637" x2="96.266" y2="13.656" width="1.27" layer="16"/>
 <wire x1="130.937" y1="27.8765" x2="130.937" y2="27.4955" width="1.27" layer="16"/>
 <wire x1="130.937" y1="27.4955" x2="127.889" y2="24.4475" width="1.27" layer="16"/>
-<wire x1="99.247" y1="21.9405" x2="99.247" y2="22.666" width="1.27" layer="16"/>
-<wire x1="99.247" y1="22.666" x2="101.0285" y2="24.4475" width="1.27" layer="16"/>
 <wire x1="135.7025" y1="11.557" x2="135.7025" y2="14.735" width="0.4064" layer="16"/>
 <wire x1="135.7025" y1="14.735" x2="135.763" y2="14.7955" width="0.4064" layer="16"/>
@@
 <wire x1="143.637" y1="34.3535" x2="143.51" y2="34.2265" width="0.3048" layer="1"/>
 <wire x1="143.51" y1="34.2265" x2="144.2085" y2="34.2265" width="0.3048" layer="1"/>
+<contactref element="TR1" pad="11"/>
+<wire x1="99.247" y1="21.9405" x2="99.247" y2="16.637" width="1.27" layer="16"/>
+<wire x1="101.747" y1="21.9405" x2="99.247" y2="21.9405" width="1.27" layer="16"/>
+<wire x1="101.747" y1="21.9405" x2="101.747" y2="22.9435" width="1.27" layer="16"/>
+<wire x1="101.747" y1="22.9435" x2="103.251" y2="24.4475" width="1.27" layer="16"/>
 </signal>
 <signal name="S2_DOT_OUT">
@@
 <vertex x="134.874" y="42.8625"/>
 </polygon>
-<contactref element="TR1" pad="11"/>
 <via x="128.27" y="41.8465" extent="1-16" drill="0.4" shape="octagon"/>
-<wire x1="101.747" y1="21.9405" x2="101.747" y2="23.769" width="0.762" layer="1"/>
-<wire x1="111.76" y1="33.782" x2="101.747" y2="23.769" width="0.762" layer="1"/>
 <wire x1="128.27" y1="41.8465" x2="128.27" y2="40.7695" width="0.6096" layer="16"/>
 <wire x1="128.27" y1="40.7695" x2="128.2725" y2="40.767" width="0.6096" layer="16"/>
-<wire x1="111.76" y1="33.782" x2="119.253" y2="33.782" width="0.762" layer="1"/>
-<wire x1="119.253" y1="33.782" x2="121.9835" y2="36.5125" width="0.762" layer="1"/>
-<wire x1="121.9835" y1="36.5125" x2="126.5555" y2="36.5125" width="0.762" layer="1"/>
-<wire x1="126.5555" y1="36.5125" x2="126.619" y2="36.576" width="0.762" layer="1"/>
+<contactref element="TR1" pad="9"/>
+<wire x1="126.8095" y1="36.703" x2="121.8565" y2="36.703" width="0.762" layer="1"/>
+<wire x1="121.8565" y1="36.703" x2="118.999" y2="33.8455" width="0.762" layer="1"/>
+<wire x1="118.999" y1="33.8455" x2="111.887" y2="33.8455" width="0.762" layer="1"/>
+<wire x1="111.887" y1="33.8455" x2="101.981" y2="23.9395" width="0.762" layer="1"/>
+<wire x1="101.981" y1="23.9395" x2="98.746" y2="23.9395" width="0.762" layer="1"/>
+<wire x1="98.746" y1="23.9395" x2="96.747" y2="21.9405" width="0.762" layer="1"/>
 </signal>
 <signal name="N$133">
@@
 <contactref element="C22" pad="2"/>
 <contactref element="TR1" pad="12"/>
-<contactref element="TR1" pad="9"/>
 <wire x1="104.247" y1="21.9405" x2="104.247" y2="23.729" width="1.27" layer="1"/>
 <wire x1="115.9735" y1="28.8925" x2="109.4105" y2="28.8925" width="1.27" layer="1"/>
 <wire x1="109.4105" y1="28.8925" x2="104.247" y2="23.729" width="1.27" layer="1"/>
-<wire x1="104.247" y1="21.9405" x2="104.247" y2="21.062" width="0.762" layer="1"/>
-<wire x1="104.247" y1="21.062" x2="103.505" y2="20.32" width="0.762" layer="1"/>
-<wire x1="103.505" y1="20.32" x2="97.7265" y2="20.32" width="0.762" layer="1"/>
-<wire x1="97.7265" y1="20.32" x2="96.747" y2="21.2995" width="0.762" layer="1"/>
-<wire x1="96.747" y1="21.9405" x2="96.747" y2="21.2995" width="0.762" layer="1"/>
 <wire x1="115.9735" y1="28.8925" x2="115.9735" y2="29.378" width="0.508" layer="1"/>
 <wire x1="115.9735" y1="29.378" x2="115.8875" y2="29.464" width="0.508" layer="1"/>

Commit message: BOM update
Parts:
- D10, D16, D19: device EEZ_Lib1:TO252 -> EEZ_Lib1:TO252-L
- moved C68 4.76 mm to (144.2, 6.79)
- moved C69 4.76 mm to (134.3, 6.79)
- moved Q7 2.54 mm to (46.9, 10.4)
- moved JP3 2.11 mm to (139.3, 14.5)
- moved D19 1.02 mm to (28.8, 52.8)
- moved D10 0.76 mm to (56.1, 67.2)
- moved X4 0.40 mm to (142.0, 9.40)
- moved C62 0.25 mm to (139.3, 6.79)
- moved C61 0.25 mm to (139.3, 11.8)
- moved SH3 0.25 mm to (53.7, 2.60)
Routing:
- net 0V: track 683.1 -> 701.4 mm
- net PE: track 230.8 -> 225.2 mm
- net CLAMP_C: track 58.0 -> 60.4 mm
- net S1_DOT_OUT: track 24.1 -> 22.4 mm, vias 27 -> 18
- net L_PULL: track 69.6 -> 68.0 mm
- net N$31: track 1.79 -> 2.93 mm
- net PREG_OUT+: track 59.6 -> 58.5 mm
- net GND: track 181.9 -> 181.3 mm

Commit message: small fixes
Parts:
- C78: value 4u7 -> N.C.
- JP3: value JP3-CUT -> 0R-JUMPA; device EEZ_Lib1:JP3-CUT -> jump-0r-smd:A0R-JMP
- Q5, Q6: value IPW60R125P6XKSA1 -> IPW60R120P7
- R49, R53: value 33R -> 10R
- R50: value 30K -> 15K
- R71: value 47K -> N.C.; device rcl:R0805 -> rcl:R2512
- R98: value 51K -> 47K
- X2: value 22-05-7085 -> 22-05-7095
- moved C67 5.97 mm to (81.4, 4.13)
- moved R71 5.85 mm to (128.9, 6.35), flipped to the top
- moved C64 2.92 mm to (123.5, 9.84)
- moved R67 2.92 mm to (123.5, 4.89)
- moved R12 2.11 mm to (121.3, 56.0), flipped to the top
- moved R8 1.03 mm to (120.6, 59.1), turned to 180 degrees
- moved C10 0.44 mm to (137.5, 17.0)
- moved C11 0.44 mm to (131.1, 18.4)
- moved C13 0.44 mm to (126.3, 16.9)
- moved L4 0.44 mm to (122.4, 16.8)
- moved L2 0.44 mm to (137.4, 20.9)
- moved D28 0.38 mm to (142.1, 24.1)
- turned JP3 to 90 degrees
Connections:
- net +12V renamed +14V
- net U_MON renamed U_CTRL
- net 12V_COMM: now also JP3.2; no longer JP3.COM
- net GND: now also JP3.3; no longer JP3.NO
- net PREG_OUT+: now also JP3.1; no longer JP3.NC
Routing:
- net PE: track 225.2 -> 219.4 mm
- net VIPER+: track 38.9 -> 36.3 mm
- net GND: track 181.3 -> 182.0 mm, vias 19 -> 23
- net N$49: track 2.91 -> 3.51 mm, vias 1 -> 0
- net N$60: track 3.25 -> 3.69 mm, vias 0 -> 1
- net PREG_OUT+: track 58.5 -> 58.6 mm, vias 5 -> 4
Other:
- board text added: "4 U_CTRL-"
- board text added: "5 U_CTRL+ (max. 2.5V)"
- board text added: "Okrenuti C57 !!!"
- board text added: "R41 povecati na 1K8?"
- board text removed: "4 U_MON-"
- board text removed: "5 U_MON+ (max. 2.5V)"
