File: Eagle files/EEZ CF-DIC block diagram r5B7.sch (EAGLE design)
At the start: 1 part

Commit message: BOM update for #7, #8
Other:
- note added: "AC filter & fuse Rectifier + Cbulk"
- note removed: "AC input filter Rectifier + Cbulk"
Changed lines of the file:
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@@
 <wire x1="22.86" y1="66.04" x2="0" y2="66.04" width="0.4064" layer="104"/>
 <wire x1="0" y1="66.04" x2="0" y2="76.2" width="0.4064" layer="104"/>
-<text x="11.43" y="71.12" size="1.778" layer="104" align="center">AC input filter
+<text x="11.43" y="71.12" size="1.778" layer="104" align="center">AC filter &amp; fuse
 Rectifier + Cbulk</text>
 <text x="27.94" y="84.455" size="1.4224" layer="109">DC_BUS</text>
