File: Mechanical/CF-DIC enclosure r5B6.brd (EAGLE design)
At the start: 0 parts

Commit message: small fixes
Other:
- board text added: "CF-DIC section U-shape heatsink (3 mm Alu)"
- board text added: "Chasis plate: 1 mm iron or aluminum"
- board text added: "HV buck section heatsink (5 mm Alu)"
- board text added: "Hole for M3 countersink"
- board text added: "Holes for M3 countersink"
- board text removed: "3.2 - 3.5 mm countersink"
- board text removed: "Chasis plate: 0.75 to 1 mm iron or aluminum"
- board text removed: "Cu-tape"
- board text removed: "PP section L-profile heatsink (3 mm Alu)"
